File: mukumiDevice/power_comtroller.brd (EAGLE design)
At the start: 160 x 100 mm, 46 parts, among them IC5 ATMEGA328-20P

Commit message: removed arduino and layout board
Parts:
- removed C15, C42: (no value), rcl:C0805
- removed C26, C27, C28: (no value), rcl:C2012
- removed IC5: ATMEGA328-20P, atmega328:DIL28-3
- removed JP1: (no value), pinhead:2X03
- removed JP3, JP6: (no value), pinhead:1X03
- removed L3: (no value), rcl:L2825P
- removed P1: (no value), Voltage Regulator:SOT-89
- removed Q2: (no value), special:QS
- removed R23: (no value), rcl:R2012
- removed S2: DTSM-6, switch-tact:DTSM-6
- removed SJ1, SJ10, SJ2, SJ20, SJ3, SJ7: (no value), jumper:SJ
- removed SV2: (no value), con-lstb:MA06-1
- added 0, R1: 1k, rcl:0204/7
- added C1, C11, C12, C4: (no value), rcl:153CLV-0810
- added C16, C17, C18, C19, C20, C21, C22, C23: (no value), rcl:D/7343-31W
- added IC1: LM317MSTT3, v-reg:SOT223
- added JP4, JP5: (no value), pinhead:1X03
- added SJ12: (no value), jumper:SJ
- added U$1: NJM2884, torex:SOT89-5
- C2, C3: device rcl:153CLV-0807 -> rcl:153CLV-0810
- C24: value (none) -> 0.33; device rcl:C0402 -> rcl:C025-024X044
- C25: value (none) -> 0.33; device rcl:C1206 -> rcl:C025-024X044
- C5, C6: device rcl:TT2D6 -> rcl:153CLV-0810
- C7, C8: value (none) -> 10u; device rcl:C025-030X050 -> rcl:E1,8-4
- L2: value (none) -> CDRH125; device rcl:L3225P -> inductor-sumida:CDRH125
- L4, L5: value CDRH127/LD -> CDRH6D28; device inductor-sumida:CDRH127/LD -> inductor-sumida:CDRH6D
- L7: value CDRH6D28 -> CDRH4D18; device inductor-sumida:CDRH6D -> inductor-sumida:CDRH4D18
- L9: value CDRH6D28 -> (none); device inductor-sumida:CDRH6D -> rcl:L2825P
- moved C24 198.8 mm to (102.9, 27.9), turned to 180 degrees
- moved SJ19 174.4 mm to (76.2, 44.5)
- moved SJ18 171.1 mm to (76.2, 39.4)
- moved L1 170.4 mm to (86.4, 44.5)
- moved SJ17 168.4 mm to (76.2, 33.0)
- moved L9 148.5 mm to (86.4, 39.4)
- moved L2 138.1 mm to (87.6, 20.3)
- moved L7 137.2 mm to (86.4, 33.0)
- moved SJ5 137.0 mm to (77.5, 20.3)
- moved C25 135.8 mm to (99.1, 30.5), turned to 180 degrees
- moved C8 132.5 mm to (97.8, 49.5), turned to 180 degrees
- moved C7 131.7 mm to (99.1, 34.3), turned to 180 degrees
- moved C6 128.5 mm to (49.5, 38.1), turned to 270 degrees
- moved SJ4 124.6 mm to (83.8, 48.3)
- moved C5 99.4 mm to (29.2, 38.1), turned to 270 degrees
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Connections:
- removed net +5V: C6.+, C8.1, JP3.3, L4.2, L6.2, L7.2
- removed net -5V: C3.+, C42.1, JP3.1, L5.2, L8.2, L9.2
- removed net 5V: SV2.4
- removed net CS: IC5.12
- removed net DTR: C28.1, SV2.1
- removed net IO_UPDATE: IC5.13
- removed net MASTER_RESET: IC5.11
- removed net N$17: L8.1, SJ8.2
- removed net N$21: IC5.19, JP1.3, SJ3.1
- removed net N$22: C26.2, IC5.10, Q2.1
- removed net N$24: C27.2, IC5.9, Q2.2
- removed net N$35: IC5.23, JP6.3
- removed net N$36: IC5.24, JP6.2
- removed net N$37: IC5.25, JP6.1
- removed net N$66: IC5.18, JP1.1, SJ2.1
- removed net N$73: IC5.17, JP1.4, SJ1.1
- removed net N$74: IC5.16
- removed net N$75: IC5.15
- removed net N$77: SJ2.2
- removed net N$8: C28.2, IC5.1, JP1.5, R23.1, S2.1, S2.2
- removed net RXD_MC: IC5.2, SV2.3
- removed net SCLK: SJ3.2
- removed net SDIO0: SJ1.2
- removed net TXD_MC: IC5.3, SV2.2
- new net 1.8V: C8.+, IC1.4
- new net F1: C22.+, C5.+, L6.1, SJ12.2
- new net F1-: C16.+, C2.+, L8.1, SJ9.2
- new net F2: C12.+, C20.+, L5.1, SJ8.2
- new net F2-: C18.+, C4.+, L4.1, SJ6.2
- new net N$1: C23.+, C6.+, JP5.1, L6.2
- new net N$7: C11.+, C21.+, JP4.3, L5.2
- net +BATTERY: now also SJ5.1; no longer SJ20.1
- net +REG: now also SJ12.1, SJ8.1; no longer C5.+, C7.1, SJ20.2, SJ5.1, SJ6.1, SJ7.1
- net -REG: now also SJ6.1; no longer C15.1, C2.+, SJ10.1, SJ8.1
- net 3.3V_MC: now also C7.+, IC1.3, U$1.4; no longer IC5.20, IC5.7, JP1.2, P1.3, R23.2, SV2.5
- net DGND: now also C7.-, C8.-, IC1.1, U$1.2; no longer C26.1, C27.1, IC5.22, IC5.8, JP1.6, P1.1, S2.3, S2.4, SV2.6
- net GND: now also C1.-, C11.-, C12.-, C16.-, C17.-, C18.-, C19.-, C20.-, C21.-, C22.-, C23.-, C4.-, JP4.2, JP5.2; no longer C15.2, C42.2, C7.2, C8.2, JP3.2
- net N$19: now also 0.1, L7.2, L9.2; no longer C24.1, L3.2, P1.2
- net N$2: now also R1.2, U$1.1; no longer L7.1, SJ7.2
- net N$29: now also L7.1; no longer L3.1
- net N$3: now also C1.+, C19.+, JP4.1, L4.2; no longer L4.1, SJ6.2
- net N$38: now also L9.1; no longer L2.1
- net N$4: now also L2.1; no longer L6.1
- net N$5: now also C17.+, C3.+, JP5.3, L8.2; no longer L9.1, SJ10.2
- net N$6: now also 0.2, C24.1, R1.1, U$1.5; no longer L5.1, SJ9.2
Routing:
- net +BATTERY: track 0.00 -> 97.6 mm
- net DGND: track 0.00 -> 50.6 mm
- net -REG: track 0.00 -> 47.7 mm
- net N$19: track 0.00 -> 44.1 mm
- net GND: track 0.00 -> 35.9 mm
- net N$1: track 0.00 -> 31.4 mm
- net N$5: track 0.00 -> 30.8 mm
- net N$3: track 0.00 -> 29.0 mm
- net N$7: track 0.00 -> 29.0 mm
- net 3.3V_MC: track 0.00 -> 29.0 mm
- net F2: track 0.00 -> 26.9 mm
- net F2-: track 0.00 -> 26.5 mm
- net +REG: track 0.00 -> 23.1 mm
- net F1-: track 0.00 -> 22.7 mm
- net F1: track 0.00 -> 22.7 mm
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- added copper zone on layer 1, net DGND
- added copper zone on layer 1, net GND
Other:
- board size 160 x 100 mm -> 110.5 x 56.8 mm
