File: mukumiDevice/power_comtroller.sch (EAGLE design)
At the start: 46 parts, among them IC5 ATMEGA328-20P

Commit message: addAnalogPowerFilter
Parts:
- removed C15, C42: (no value), rcl:C-EUC0805
- removed L3: (no value), rcl:L-USL2825P
- removed P1: (no value), Voltage Regulator:XC6206SOT-89
- added C1, C11, C12, C4: (no value), rcl:CPOL-EUTT2D6
- added C16, C17, C18, C19, C20, C21, C22, C23: (no value), rcl:CPOL-EUD/7343-31W
- added IC1: LM317MSTT3, v-reg:LM317MSTT3
- added R1: 1k, rcl:R-EU_0204/2V
- added SJ11, SJ12, SJ13: (no value), jumper:SJ
- added U$1: NJM2884, torex:NJM2884
- C24, C25: value (none) -> 0.33
- C7, C8: value (none) -> 10u; device rcl:C-EU025-030X050 -> rcl:C-EUC0402
- L2: value (none) -> CDRH125; device rcl:L-USL3225P -> inductor-sumida:CDRH125
- L4, L5: value CDRH127/LD -> CDRH6D28; device inductor-sumida:CDRH127/LD -> inductor-sumida:CDRH6D28
- L9: value CDRH6D28 -> (none); device inductor-sumida:CDRH6D28 -> rcl:L-USL2825P
Connections:
- removed net N$17: L8.1, SJ8.2
- removed net N$6: L5.1, SJ9.2
- new net 1.8V: C8.1, IC1.OUT
- new net F1: C22.+, C5.+, L6.1, SJ12.2
- new net F1-: C16.+, C2.+, L8.1, SJ9.2
- new net F2: C12.+, C20.+, L5.1, SJ8.2
- new net F2-: C18.+, C4.+, L4.1, SJ6.2
- new net N$1: C23.+, C6.+, L6.2, SJ11.1
- new net N$7: C11.+, C21.+, L5.2, SJ13.1
- net +5V: now also SJ11.2, SJ13.2; no longer C6.+, C8.1, L4.2, L6.2, L7.2
- net +BATTERY: now also SJ5.1
- net +REG: now also SJ12.1, SJ8.1; no longer C5.+, C7.1, SJ5.1, SJ6.1, SJ7.1
- net -5V: now also SJ10.2, SJ7.2; no longer C3.+, C42.1, L5.2, L8.2, L9.2
- net -REG: now also SJ6.1; no longer C15.1, C2.+, SJ10.1, SJ8.1
- net 3.3V_MC: now also C7.1, IC1.IN, U$1.VOUT; no longer P1.OUT
- net DGND: now also C7.2, C8.2, IC1.ADJ, U$1.GND; no longer P1.VSS
- net GND: now also C1.-, C11.-, C12.-, C16.-, C17.-, C18.-, C19.-, C20.-, C21.-, C22.-, C23.-, C4.-; no longer C15.2, C42.2, C7.2, C8.2
- net N$19: now also L7.2, L9.2, R1.1, U$1.VIN; no longer L3.2, P1.IN
- net N$2: now also R1.2, U$1.CE; no longer L7.1, SJ7.2
- net N$29: now also L7.1; no longer L3.1
- net N$3: now also C1.+, C19.+, L4.2, SJ7.1; no longer L4.1, SJ6.2
- net N$38: now also L9.1; no longer L2.1
- net N$4: now also L2.1; no longer L6.1
- net N$5: now also C17.+, C3.+, L8.2, SJ10.1; no longer L9.1, SJ10.2
Other:
- moved on the sheet: C24, C25, C7, C8, L2, L4, L5, L7, L9, SJ10, SJ5, SJ6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

Commit message: removed arduino and layout board
Parts:
- removed C26, C27, C28: (no value), rcl:C-EUC2012
- removed IC5: ATMEGA328-20P, atmega328:ATMEGA328-20P
- removed JP1: (no value), pinhead:PINHD-2X3
- removed JP3, JP6: (no value), pinhead:PINHD-1X3
- removed Q2: (no value), special:XTAL/S
- removed R23: (no value), rcl:R-EU_R2012
- removed S2: DTSM-6, switch-tact:DTSM-6
- removed SJ1, SJ10, SJ11, SJ13, SJ2, SJ20, SJ3, SJ7: (no value), jumper:SJ
- removed SV2: (no value), con-lstb:MA06-1
- added 0: 1k, rcl:R-EU_0204/7
- added JP4, JP5: (no value), pinhead:PINHD-1X3
- C1, C11, C12, C4, C5, C6: device rcl:CPOL-EUTT2D6 -> rcl:CPOL-EU153CLV-0810
- C2, C3: device rcl:CPOL-EU153CLV-0807 -> rcl:CPOL-EU153CLV-0810
- C24: device rcl:C-EUC0402 -> rcl:C-EU025-024X044
- C25: device rcl:C-EUC1206 -> rcl:C-EU025-024X044
- C7, C8: device rcl:C-EUC0402 -> rcl:CPOL-USE1.8-4
- L7: value CDRH6D28 -> CDRH4D18; device inductor-sumida:CDRH6D28 -> inductor-sumida:CDRH4D18
- R1: device rcl:R-EU_0204/2V -> rcl:R-EU_0204/7
Connections:
- removed net +5V: JP3.3, SJ11.2, SJ13.2
- removed net -5V: JP3.1, SJ10.2, SJ7.2
- removed net 5V: SV2.4
- removed net CS: IC5.(PCI22/AIN0OC0A)PD6
- removed net DTR: C28.1, SV2.1
- removed net IO_UPDATE: IC5.(PCI23/AIN1)PD7
- removed net MASTER_RESET: IC5.(PCI21/T1/OC0B)PD5
- removed net N$21: IC5.(PCI5/SCK)PB5, JP1.3, SJ3.1
- removed net N$22: C26.2, IC5.PB7(XTAL2/TOSC2/PCI7), Q2.1
- removed net N$24: C27.2, IC5.PB6(XTAL1/TOSC1/PCI6), Q2.2
- removed net N$35: IC5.(PCI8/ADC0)PC0, JP6.3
- removed net N$36: IC5.(PCI9/ADC1)PC1, JP6.2
- removed net N$37: IC5.(PCI10/ADC2)PC2, JP6.1
- removed net N$66: IC5.(PCI4/MISO)PB4, JP1.1, SJ2.1
- removed net N$73: IC5.(PCI3/MOSI/OC2A)PB3, JP1.4, SJ1.1
- removed net N$74: IC5.(PCI2/SS/OC1B)PB2
- removed net N$75: IC5.(PCI1/OC1A/OC1S)PB1
- removed net N$77: SJ2.2
- removed net N$8: C28.2, IC5.PC6(/RESET/PCI14), JP1.5, R23.1, S2.1, S2.2
- removed net RXD_MC: IC5.(PCI16/RXD)PD0, SV2.3
- removed net SCLK: SJ3.2
- removed net SDIO0: SJ1.2
- removed net TXD_MC: IC5.(PCI17/TXD)PD1, SV2.2
- new net N$6: 0.2, C24.1, R1.1, U$1.VIN
- net +BATTERY: no longer SJ20.1
- net +REG: no longer SJ20.2
- net 1.8V: now also C8.+; no longer C8.1
- net 3.3V_MC: now also C7.+; no longer C7.1, IC5.AVCC, IC5.VCC, JP1.2, R23.2, SV2.5
- net DGND: now also C7.-, C8.-; no longer C26.1, C27.1, C7.2, C8.2, IC5.AGND, IC5.GND, JP1.6, S2.3, S2.4, SV2.6
- net GND: now also JP4.2, JP5.2; no longer JP3.2
- net N$1: now also JP5.1; no longer SJ11.1
- net N$19: now also 0.1; no longer C24.1, R1.1, U$1.VIN
- net N$3: now also JP4.1; no longer SJ7.1
- net N$5: now also JP5.3; no longer SJ10.1
- net N$7: now also JP4.3; no longer SJ13.1
