File: mukumiDevice/mukumi_ad9834_wearable.brd (EAGLE design)
At the start: 54 x 90 mm, 143 parts, among them IC1A1 1k, IC1A1,1 1k, IC1A3'1 560, IC1B1 1k, IC1B2 1k, IC1B6,1 2k, IC2A1,1 5.1k, IC2A3 20k, IC2A3,2 20k, IC2A4 5.1k, IC2B1 20k, IC2B2 5.1k, IC2B3 20k, IC2B6,1 5.1k, IC3A2 56, IC3B1 56, IC4 TL072D, IC4A1 560, IC4A2,2 560, IC4B1 62a, IC4B2 560, IC4B6,1 560a, IC4B6,10 560a, IC4B6,11 560a, IC4B6,12 560a, IC4B6,13 560a, IC4B6,2 560a, IC4B6,3 560a, IC4B6,4 560a, IC4B6,5 560a, IC4B6,6 560a, IC4B6,7 560a, IC4B6,8 560a, IC4B6,9 560a, Q2 FA-20H, U1 AD9834, U2 AD9834

Commit message: AGNDとDGNDの接続の問題
Parts:
- removed QG1: (no value), crystal:DIL08-4
- added U$8: SG8002LB, sg-8002:SG-8002LB
Connections:
- net AGND: now also SV1.3
- net GND: now also U$8.P$2; no longer QG1.2, SV1.3
- net N$8: now also U$8.P$3; no longer QG1.3
- net VDD: now also U$8.P$4; no longer QG1.4
Routing:
- net GND: track 215.6 -> 211.3 mm
Changed lines of the file:
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@@
 <element name="U1" library="ad9834" package="TSSOP20" value="AD9834" x="46.101" y="-18.415" rot="MR270"/>
 <element name="U2" library="ad9834" package="TSSOP20" value="AD9834" x="46.101" y="-36.957" rot="MR270"/>
-<element name="QG1" library="crystal" package="DIL08-4" value="" x="68.326" y="-25.146" rot="R180">
-<attribute name="MF" value="" x="49.276" y="-20.066" size="1.778" layer="27" rot="R180" display="off"/>
-<attribute name="MPN" value="SG531P16MHZ" x="49.276" y="-20.066" size="1.778" layer="27" rot="R180" display="off"/>
-<attribute name="OC_FARNELL" value="unknown" x="49.276" y="-20.066" size="1.778" layer="27" rot="R180" display="off"/>
-<attribute name="OC_NEWARK" value="01M8837" x="49.276" y="-20.066" size="1.778" layer="27" rot="R180" display="off"/>
-</element>
 <element name="R2" library="rcl" package="R0402" value="6.8k" x="47.117" y="-32.004"/>
 <element name="C9" library="rcl" package="C0402K" value="0.1u" x="47.117" y="-29.845"/>
@@
 <element name="C35" library="rcl" package="C0402K" value="0.1u" x="55.88" y="-9.271" rot="R270"/>
 <element name="C36" library="rcl" package="C0402K" value="0.01u" x="66.421" y="-8.128" rot="R90"/>
+<element name="U$8" library="sg-8002" package="SG-8002LB" value="SG8002LB" x="0.5" y="-66.6"/>
 </elements>
 <signals>
@@
 <contactref element="IC4B1" pad="1"/>
 <contactref element="IC4B2" pad="1"/>
-<contactref element="SV1" pad="3"/>
 <contactref element="C,IC2A2" pad="2"/>
 <contactref element="C,IC2A4" pad="2"/>
@@
 <wire x1="25.704" y1="53.386" x2="25.738" y2="53.42" width="0.254" layer="16"/>
 <wire x1="46.49" y1="60.34" x2="47.12" y2="60.34" width="0.254" layer="1"/>
-<wire x1="47.12" y1="60.34" x2="50.16" y2="63.38" width="0.254" layer="1"/>
 <wire x1="45.14" y1="53.3" x2="45.14" y2="50.59" width="0.254" layer="16"/>
 <wire x1="45.14" y1="50.59" x2="44.96" y2="50.41" width="0.254" layer="16"/>
@@
 <contactref element="U1" pad="7"/>
 <contactref element="U2" pad="7"/>
-<contactref element="QG1" pad="2"/>
 <contactref element="C32" pad="2"/>
 <contactref element="C13" pad="2"/>
@@
 <contactref element="R19" pad="2"/>
 <contactref element="C34" pad="1"/>
+<contactref element="U$8" pad="P$2"/>
 <wire x1="42.43" y1="59.19" x2="46.49" y2="60.34" width="0" layer="19" extent="1-1"/>
 <wire x1="45.14" y1="53.3" x2="42.43" y2="59.19" width="0" layer="19" extent="1-16"/>
@@
 <wire x1="45.227" y1="-27.686" x2="48.895" y2="-25.796" width="0" layer="19" extent="1-1"/>
 <wire x1="59.309" y1="-18.253" x2="49.196" y2="-19.215" width="0" layer="19" extent="1-16"/>
-<wire x1="64.516" y1="-21.336" x2="59.309" y2="-18.253" width="0" layer="19" extent="1-1"/>
-<wire x1="66.548" y1="-18.761" x2="64.516" y2="-21.336" width="0" layer="19" extent="1-1"/>
+<wire x1="66.548" y1="-18.761" x2="59.309" y2="-18.253" width="0" layer="19" extent="1-1"/>
 <wire x1="49.196" y1="-37.757" x2="45.227" y2="-27.686" width="0" layer="19" extent="1-16"/>
 <wire x1="52.324" y1="-44.211" x2="49.196" y2="-37.757" width="0" layer="19" extent="1-16"/>
@@
 <wire x1="65.624" y1="-34.29" x2="60.071" y2="-40.351" width="0" layer="19" extent="1-1"/>
 <wire x1="69.631" y1="-36.576" x2="65.624" y2="-34.29" width="0" layer="19" extent="1-1"/>
+<wire x1="1.77" y1="-67.7" x2="46.228" y2="-47.356" width="0" layer="19" extent="1-1"/>
 </signal>
 <signal name="N$26">
@@
 </signal>
 <signal name="N$8">
-<contactref element="QG1" pad="3"/>
 <contactref element="U1" pad="8"/>
 <contactref element="U2" pad="8"/>
-<wire x1="49.196" y1="-19.865" x2="64.516" y2="-28.956" width="0" layer="19" extent="16-16"/>
-<wire x1="49.196" y1="-38.407" x2="64.516" y2="-28.956" width="0" layer="19" extent="16-16"/>
+<contactref element="U$8" pad="P$3"/>
+<wire x1="49.196" y1="-38.407" x2="1.77" y2="-65.5" width="0" layer="19" extent="1-16"/>
+<wire x1="49.196" y1="-19.865" x2="49.196" y2="-38.407" width="0" layer="19" extent="16-16"/>
 </signal>
 <signal name="VDD">
-<contactref element="QG1" pad="4"/>
 <contactref element="C32" pad="1"/>
-<wire x1="70.831" y1="-36.576" x2="72.136" y2="-28.956" width="0" layer="19" extent="1-1"/>
+<contactref element="U$8" pad="P$4"/>
+<wire x1="70.831" y1="-36.576" x2="-0.77" y2="-65.5" width="0" layer="19" extent="1-1"/>
 </signal>
 <signal name="N$9">
@@
 <contactref element="R18" pad="2"/>
 <contactref element="C35" pad="1"/>
-<wire x1="55.88" y1="-8.671" x2="60.071" y2="-9.941" width="0" layer="19" extent="1-1"/>
-<wire x1="52.451" y1="-8.367" x2="55.88" y2="-8.671" width="0" layer="19" extent="1-1"/>
+<contactref element="SV1" pad="3"/>
+<wire x1="52.451" y1="-8.367" x2="50.16" y2="63.38" width="0" layer="19" extent="1-1"/>
 <wire x1="49.53" y1="-8.417" x2="52.451" y2="-8.367" width="0" layer="19" extent="1-1"/>
+<wire x1="55.88" y1="-8.671" x2="52.451" y2="-8.367" width="0" layer="19" extent="1-1"/>
+<wire x1="60.071" y1="-9.941" x2="55.88" y2="-8.671" width="0" layer="19" extent="1-1"/>
 <wire x1="43.196" y1="-16.615" x2="49.53" y2="-8.417" width="0" layer="19" extent="1-16"/>
-<wire x1="41.29" y1="-23.749" x2="43.196" y2="-16.615" width="0" layer="19" extent="16-16"/>
+<wire x1="41.29" y1="-23.749" x2="43.196" y2="-16.615" width="0" layer="19" extent="1-16"/>
 <wire x1="46.517" y1="-29.845" x2="41.29" y2="-23.749" width="0" layer="19" extent="1-1"/>
 <wire x1="46.467" y1="-32.004" x2="46.517" y2="-29.845" width="0" layer="19" extent="1-1"/>
-<wire x1="43.196" y1="-35.157" x2="46.467" y2="-32.004" width="0" layer="19" extent="16-16"/>
+<wire x1="43.196" y1="-35.157" x2="46.467" y2="-32.004" width="0" layer="19" extent="1-16"/>
 <wire x1="51.816" y1="-26.705" x2="46.517" y2="-29.845" width="0" layer="19" extent="1-1"/>
 <wire x1="58.166" y1="-28.356" x2="51.816" y2="-26.705" width="0" layer="19" extent="1-1"/>
-<wire x1="40.64" y1="-45.862" x2="43.196" y2="-35.157" width="0" layer="19" extent="16-16"/>
+<wire x1="40.64" y1="-45.862" x2="43.196" y2="-35.157" width="0" layer="19" extent="1-16"/>
 <wire x1="36.357" y1="-49.784" x2="40.64" y2="-45.862" width="0" layer="19" extent="1-1"/>
 <wire x1="36.357" y1="-53.086" x2="36.357" y2="-49.784" width="0" layer="19" extent="1-1"/>

Commit message: brdにdds配置・配線（未完）
Parts:
- removed C43, C50: 22p, rcl:C0402
- removed JP1, JP11, JP5, JP51, JP52, JP53: (no value), pinhead:1X01
- removed Q2: FA-20H, crystal:FA-20H
- removed R25, R27, R31, R32, R33, R34, R35, R36: 100, rcl:R0402
- removed U$8: SG8002LB, sg-8002:SG-8002LB
- added C23, C40: 0.47u, rcl:C0805
- added C37, C39: 3p, rcl:C0402
- added R16, R26: 3.3k, rcl:R0402
- added R17, R22: 22k, rcl:R0402
- added R21, R24: 2.7k, rcl:R0402
- added U$9: SG710, SG:SG710
- C10, C13, C14, C16, C17, C20, C21, C26, C27, C28, C31, C32, C33, C34, C35, C36, C9: device rcl:C0402K -> rcl:C0402
- moved R4 116.9 mm to (9.41, 55.8), flipped to the bottom, turned to 0 degrees
- moved C21 110.4 mm to (19.8, 55.9), turned to 90 degrees
- moved R6 108.5 mm to (17.6, 55.7), turned to 0 degrees
- moved C32 106.5 mm to (4.78, 47.4), turned to 270 degrees
- moved C34 103.7 mm to (9.75, 50.9), turned to 0 degrees
- moved C27 102.5 mm to (9.78, 52.1), turned to 180 degrees
- moved R19 102.5 mm to (11.3, 48.1)
- moved R8 99.9 mm to (17.6, 47.7), flipped to the bottom, turned to 0 degrees
- moved R5 98.9 mm to (13.7, 47.4), turned to 0 degrees
- moved C14 98.4 mm to (10.6, 55.3), turned to 180 degrees
- moved C17 98.3 mm to (17.6, 46.6), flipped to the bottom
- moved C26 96.1 mm to (10.2, 54.3), turned to 180 degrees
- moved R12 95.4 mm to (18.2, 47.5), turned to 180 degrees
- moved R2 93.6 mm to (14.5, 55.7), turned to 180 degrees
- moved U2 93.3 mm to (16.0, 51.3), flipped to the top
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Connections:
- net N$42 renamed DDS_OUT1B
- net N$65 renamed DDS_OUT2B
- removed net CH0_IOUT_1: R31.1
- removed net CH0_IOUT_2: R32.1
- removed net CH1_IOUT1: R25.1
- removed net CH1_IOUT2: R27.1
- removed net N$11: JP53.1, U1.15
- removed net N$13: C16.1, JP5.1, R9.2, U2.19
- removed net N$14: ATMEGA328.7, C50.2, Q2.3
- removed net N$15: JP51.1, U1.13, U2.13
- removed net N$16: JP11.1, U1.14, U2.14
- removed net N$18: JP52.1, U2.15
- removed net N$23: C28.1, U1.5
- removed net N$24: C31.1, U1.4
- removed net N$64: R25.2, R36.1, U$3.13
- removed net N$69: R27.2, R35.1, U$3.12
- removed net N$71: C20.1, JP1.1, R7.2, U1.19
- removed net N$72: C14.2, C26.1, U2.4
- removed net N$73: C27.1, U2.5
- removed net SDIO0: SJ2.1
- new net DDS_OUT1: C16.1, C23.1, R9.2, U2.19
- new net DDS_OUT2: C20.1, C40.1, R7.2, U1.19
- new net FSYNC1: U2.15
- new net FSYNC2: U1.15
- new net N$39: R24.1, U$3.13
- new net N$91: C39.1, R22.1, R26.1, U$3.12
- new net N$93: C40.2, R26.2
- new net SDATA: SJ2.1, U1.13, U2.13
- net +5V: no longer C36.1
- net 3.3V_DDS: now also C14.2, C26.1, C31.1, C36.1, U1.4, U2.4
- net 3.3V_MC: now also C27.1, C28.1, U1.5, U2.5
- net AGND: now also R21.2, R24.2
- net COS: now also C39.2, R22.2; no longer R35.2
- net GND: now also U$9.P$2; no longer C43.1, C50.1, R34.2, R36.2, U$8.P$2
- net N$1: now also R21.1, U$3.2; no longer ATMEGA328.8, C43.2, Q2.1
- net N$76: now also C23.2, R16.2; no longer R31.2, R34.1, U$3.2
- net N$78: now also C37.1, R16.1, R17.1; no longer R32.2, R33.1
- net N$8: now also U$9.P$3; no longer U$8.P$3
- net SCLK: now also U1.14, U2.14
- net SIN: now also C37.2, R17.2; no longer R33.2
- net VDD: now also U$9.P$4; no longer U$8.P$4
Routing:
- net GND: track 211.3 -> 266.8 mm, vias 8 -> 9
- net AGND: track 0.00 -> 24.2 mm
- net N$8: track 0.00 -> 17.3 mm, vias 0 -> 1
- net 3.3V_MC: track 0.00 -> 12.5 mm, vias 0 -> 1
- net SDATA: track 0.00 -> 11.8 mm, vias 0 -> 1
- net SCLK: track 0.00 -> 11.5 mm, vias 0 -> 1
- net SIG*SIN: track 20.2 -> 8.95 mm
- net COS: track 41.2 -> 32.5 mm, vias 2 -> 1
- net CH0_IOUT_2: track 6.87 -> 0.00 mm
- net N$69: track 6.66 -> 0.00 mm
- net DDS_OUT1: track 0.00 -> 6.64 mm
- net N$64: track 5.77 -> 0.00 mm, vias 1 -> 0
- net DDS_OUT2: track 0.00 -> 5.58 mm
- net CH0_IOUT_1: track 5.30 -> 0.00 mm, vias 1 -> 0
- net CH1_IOUT2: track 4.22 -> 0.00 mm, vias 1 -> 0
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