File: mukumiDevice/mukumi_ad9834_wearable.brd (EAGLE design)
At the start: 54 x 90 mm, 136 parts, among them IC1A1 1k, IC1A1,1 1k, IC1A3'1 560, IC1B1 1k, IC1B2 1k, IC1B6,1 2k, IC2A1,1 5.1k, IC2A3 20k, IC2A3,2 20k, IC2A4 5.1k, IC2B1 20k, IC2B2 5.1k, IC2B3 20k, IC2B6,1 5.1k, IC3A2 56, IC3B1 56, IC4 TL072D, IC4A1 560, IC4A2,2 560, IC4B1 62a, IC4B2 560, IC4B6,1 560a, IC4B6,10 560a, IC4B6,11 560a, IC4B6,12 560a, IC4B6,13 560a, IC4B6,2 560a, IC4B6,3 560a, IC4B6,4 560a, IC4B6,5 560a, IC4B6,6 560a, IC4B6,7 560a, IC4B6,8 560a, IC4B6,9 560a, U1 AD9834, U2 AD9834

Commit message: mems発振器に変更と電源周り配線修正
Parts:
- moved C24 3.41 mm to (12.7, 34.0), turned to 90 degrees
- moved C17 0.60 mm to (17.0, 46.6)
Connections:
- net AGND: now also AD633_1.2, AD633_1.4, AD633_1.7, AD633_2.2, AD633_2.4, AD633_2.7, AD633_3.2, AD633_3.4, AD633_3.7, C,IC2A1.2, C,IC2A10.1, C,IC2A11.2, C,IC2A12.1, C,IC2A13.1, C,IC2A14.1, C,IC2A15.2, C,IC2A16.1, C,IC2A17.2, C,IC2A18.1, C,IC2A2.2, C,IC2A4.2, C,IC2A5.2, C,IC2A6.2, C,IC2A7.1, C,IC2A8.1, C,IC2A9.1, C30.1, C6.1, C7.1, IC1A1.1, IC1A3'1.1, IC1B1.2, IC2A3,2.2, IC2B3.2, IC4A1.2, IC4B1.1, IC4B2.1, IC4B6,12.1, IC4B6,8.1, IC4B6,9.1
- net GND: no longer AD633_1.2, AD633_1.4, AD633_1.7, AD633_2.2, AD633_2.4, AD633_2.7, AD633_3.2, AD633_3.4, AD633_3.7, C,IC2A1.2, C,IC2A10.1, C,IC2A11.2, C,IC2A12.1, C,IC2A13.1, C,IC2A14.1, C,IC2A15.2, C,IC2A16.1, C,IC2A17.2, C,IC2A18.1, C,IC2A2.2, C,IC2A4.2, C,IC2A5.2, C,IC2A6.2, C,IC2A7.1, C,IC2A8.1, C,IC2A9.1, C30.1, C6.1, C7.1, IC1A1.1, IC1A3'1.1, IC1B1.2, IC2A3,2.2, IC2B3.2, IC4A1.2, IC4B1.1, IC4B2.1, IC4B6,12.1, IC4B6,8.1, IC4B6,9.1
Routing:
- net AGND: track 24.2 -> 174.9 mm, vias 0 -> 19
- net GND: track 275.7 -> 210.2 mm, vias 9 -> 3
- net 3.3V_MC: track 31.0 -> 55.1 mm, vias 1 -> 2
- net 3.3V_DDS: track 22.1 -> 40.5 mm, vias 1 -> 2
- net -5V: track 148.2 -> 154.5 mm
- net +5V: track 119.2 -> 124.5 mm
- net COS: track 32.5 -> 37.0 mm
- net N$91: track 0.00 -> 3.16 mm
- net SIG*SIN: track 8.95 -> 12.0 mm, vias 0 -> 1
- net SIN*SIN: track 7.23 -> 8.74 mm, vias 0 -> 1
- net SIG*COS: track 9.32 -> 10.7 mm, vias 0 -> 1
- net N$39: track 0.00 -> 1.34 mm
- net +BATTERY: track 3.46 -> 4.47 mm
