File: mukumiDevice/mukumi_ad9834_wearable.brd (EAGLE design)
At the start: 54 x 90 mm, 136 parts, among them IC1A1 1k, IC1A1,1 1k, IC1A3'1 560, IC1B1 1k, IC1B2 1k, IC1B6,1 2k, IC2A1,1 5.1k, IC2A3 20k, IC2A3,2 20k, IC2A4 5.1k, IC2B1 20k, IC2B2 5.1k, IC2B3 20k, IC2B6,1 5.1k, IC3A2 56, IC3B1 56, IC4 TL072D, IC4A1 560, IC4A2,2 560, IC4B1 62a, IC4B2 560, IC4B6,1 560a, IC4B6,10 560a, IC4B6,11 560a, IC4B6,12 560a, IC4B6,13 560a, IC4B6,2 560a, IC4B6,3 560a, IC4B6,4 560a, IC4B6,5 560a, IC4B6,6 560a, IC4B6,7 560a, IC4B6,8 560a, IC4B6,9 560a, U1 AD9834, U2 AD9834

Commit message: DDSのAGND,GNDの間違いの修正
Connections:
- net AGND: now also R6.1, R9.1; no longer R12.2, R14.1
- net GND: now also R12.2, R14.1; no longer R6.1, R9.1
Routing:
- net AGND: track 174.9 -> 168.7 mm
- net GND: track 212.2 -> 209.2 mm
Changed lines of the file:
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@@
 <contactref element="R5" pad="2"/>
 <contactref element="R8" pad="1"/>
-<contactref element="R9" pad="1"/>
 <contactref element="R7" pad="1"/>
-<contactref element="R6" pad="1"/>
 <contactref element="C27" pad="2"/>
 <contactref element="C28" pad="2"/>
@@
 <contactref element="R19" pad="2"/>
 <contactref element="C34" pad="1"/>
-<wire x1="16.929" y1="53.629" x2="16.929" y2="55.684" width="0.254" layer="1"/>
 <wire x1="13.843" y1="50.543" x2="12.906" y2="50.543" width="0.254" layer="1"/>
 <wire x1="13.95" y1="50.65" x2="13.843" y2="50.543" width="0.254" layer="1"/>
@@
 <wire x1="18.25" y1="34.3398" x2="18.25" y2="32.7" width="0.254" layer="16"/>
 <wire x1="18.25" y1="34.3398" x2="18.8014" y2="34.8912" width="0.254" layer="16"/>
-<wire x1="21.373" y1="53.427" x2="21.286" y2="53.427" width="0.254" layer="1"/>
-<wire x1="21.373" y1="53.427" x2="21.4" y2="53.4" width="0.254" layer="1"/>
 <wire x1="11.119" y1="45.776" x2="11.119" y2="45.919" width="0.254" layer="1"/>
 <wire x1="11.119" y1="45.919" x2="11.2" y2="46" width="0.254" layer="1"/>
-<wire x1="16.929" y1="55.684" x2="16.916" y2="55.684" width="0.254" layer="1"/>
-<wire x1="16.916" y1="55.684" x2="16.8" y2="55.8" width="0.254" layer="1"/>
-<wire x1="21.286" y1="53.427" x2="21.286" y2="54.2605375" width="0.254" layer="1"/>
 <wire x1="21.286" y1="54.2605375" x2="21.244" y2="54.3025375" width="0.254" layer="1"/>
 <wire x1="21.244" y1="55.656" x2="21" y2="55.9" width="0.254" layer="1"/>
@@
 <wire x1="25.11" y1="30.61" x2="25.11" y2="30.15" width="0.254" layer="16"/>
 <wire x1="25.11" y1="30.15" x2="24.07" y2="29.11" width="0.254" layer="16"/>
+<contactref element="R12" pad="2"/>
+<wire x1="17.538" y1="47.46" x2="17.54" y2="47.46" width="0.254" layer="1"/>
+<wire x1="17.54" y1="47.46" x2="17.7" y2="47.3" width="0.254" layer="1"/>
+<contactref element="R14" pad="1"/>
 <wire x1="18.03" y1="62.05" x2="16.7" y2="75.85" width="0" layer="19" extent="1-16"/>
+<wire x1="17.7" y1="47.3" x2="18.244" y2="47.672" width="0" layer="19" extent="1-16"/>
+<wire x1="16.79" y1="56.151" x2="16.929" y2="53.629" width="0" layer="19" extent="1-16"/>
 <wire x1="20.035" y1="43.165" x2="19.171725" y2="45.744" width="0" layer="19" extent="1-16"/>
 </signal>
@@
 <contactref element="R2" pad="1"/>
 <contactref element="C9" pad="1"/>
-<contactref element="R12" pad="2"/>
-<contactref element="R14" pad="1"/>
 <contactref element="C33" pad="2"/>
 <contactref element="R18" pad="2"/>
@@
 <wire x1="16.8" y1="52.2" x2="17.743" y2="53.143" width="0.254" layer="1"/>
 <via x="16.8" y="52.2" extent="1-16" drill="0.3"/>
-<wire x1="17.538" y1="51.462" x2="17.538" y2="47.46" width="0.254" layer="1"/>
 <wire x1="17.538" y1="51.462" x2="16.8" y2="52.2" width="0.254" layer="1"/>
 <wire x1="19.814" y1="56.593" x2="19" y2="56.593" width="0.254" layer="1"/>
@@
 <wire x1="15.24" y1="56.593" x2="15.133" y2="56.7" width="0.254" layer="1"/>
 <wire x1="12.669" y1="57.282" x2="12.3" y2="57.651" width="0.254" layer="16"/>
-<wire x1="16.79" y1="56.151" x2="14.7434625" y2="56.151" width="0.254" layer="16"/>
 <wire x1="14.7434625" y1="56.151" x2="13.6124625" y2="57.282" width="0.254" layer="16"/>
 <wire x1="13.6124625" y1="57.282" x2="12.669" y2="57.282" width="0.254" layer="16"/>
@@
 <wire x1="19.814" y1="56.586" x2="19.814" y2="56.593" width="0.254" layer="1"/>
 <wire x1="19.814" y1="56.586" x2="19.9" y2="56.5" width="0.254" layer="1"/>
-<wire x1="17.538" y1="47.46" x2="17.54" y2="47.46" width="0.254" layer="1"/>
-<wire x1="17.54" y1="47.46" x2="17.7" y2="47.3" width="0.254" layer="1"/>
 <wire x1="18.516" y1="46.584" x2="17.693" y2="46.584" width="0.254" layer="16"/>
 <wire x1="18.516" y1="46.584" x2="18.9" y2="46.4" width="0.254" layer="16"/>
@@
 <via x="23.9" y="58.1" extent="1-16" drill="0.3"/>
 <wire x1="19" y1="56.593" x2="19" y2="56.7" width="0.254" layer="1"/>
+<contactref element="R9" pad="1"/>
+<wire x1="21.373" y1="53.427" x2="21.286" y2="53.427" width="0.254" layer="1"/>
+<wire x1="21.373" y1="53.427" x2="21.4" y2="53.4" width="0.254" layer="1"/>
+<contactref element="R6" pad="1"/>
 <wire x1="47.12" y1="60.34" x2="50.16" y2="63.38" width="0" layer="19" extent="1-1"/>
 <wire x1="42.43" y1="59.19" x2="46.49" y2="60.34" width="0" layer="19" extent="1-1"/>
@@
 <wire x1="23.85" y1="56.9" x2="27.71" y2="55.59" width="0" layer="19" extent="1-16"/>
 <wire x1="22.377" y1="53.423" x2="23.85" y2="56.9" width="0" layer="19" extent="1-1"/>
+<wire x1="21.4" y1="53.4" x2="22.339" y2="53.423" width="0" layer="19" extent="1-1"/>
+<wire x1="18.906" y1="53.143" x2="21.286" y2="53.427" width="0" layer="19" extent="1-1"/>
+<wire x1="18.204" y1="50.415" x2="17.538" y2="51.462" width="0" layer="19" extent="1-16"/>
 <wire x1="20.983" y1="47.84" x2="23.144" y2="48.928275" width="0" layer="19" extent="1-16"/>
-<wire x1="17.7" y1="47.3" x2="17.8" y2="46.6" width="0" layer="19" extent="1-16"/>
-<wire x1="18.204" y1="50.415" x2="17.538" y2="51.462" width="0" layer="19" extent="1-16"/>
-<wire x1="16.79" y1="56.151" x2="17.743" y2="53.143" width="0" layer="19" extent="1-16"/>
+<wire x1="16.929" y1="55.684" x2="17.743" y2="53.143" width="0" layer="19" extent="1-1"/>
+<wire x1="15.133" y1="55.704" x2="16.929" y2="55.684" width="0" layer="19" extent="1-1"/>
 <wire x1="8.591" y1="50.571" x2="9.506" y2="54.266" width="0" layer="19" extent="1-16"/>
 <wire x1="43.958" y1="41.758" x2="44.09" y2="46.57" width="0" layer="19" extent="2-16"/>
