File: mukumiDevice/mukumi_ad9834_wearable.sch (EAGLE design)
At the start: 143 parts, among them IC1A1 1k, IC1A1,1 1k, IC1A3'1 560, IC1B1 1k, IC1B2 1k, IC1B6,1 2k, IC2A1,1 5.1k, IC2A3 20k, IC2A3,2 20k, IC2A4 5.1k, IC2B1 20k, IC2B2 5.1k, IC2B3 20k, IC2B6,1 5.1k, IC3A2 56, IC3B1 56, IC4 TL072D, IC4A1 560, IC4A2,2 560, IC4B1 62a, IC4B2 560, IC4B6,1 560a, IC4B6,10 560a, IC4B6,11 560a, IC4B6,12 560a, IC4B6,13 560a, IC4B6,2 560a, IC4B6,3 560a, IC4B6,4 560a, IC4B6,5 560a, IC4B6,6 560a, IC4B6,7 560a, IC4B6,8 560a, IC4B6,9 560a, Q2 FA-20H, U1 AD9834, U2 AD9834

Commit message: AGNDとDGNDの接続の問題
Parts:
- removed QG1: (no value), crystal:SG531
- added U$8: SG8002LB, sg-8002:SG8002LB
Connections:
- net AGND: now also SV1.3
- net GND: now also U$8.GND; no longer QG1.GND, SV1.3
- net N$8: now also U$8.OUT; no longer QG1.OUT
- net VDD: now also U$8.VDD; no longer QG1.VCC
Other:
- moved on the sheet: C32

Commit message: brdにdds配置・配線（未完）
Parts:
- removed C43, C50: 22p, rcl:C-EUC0402
- removed JP1, JP11, JP5, JP51, JP52, JP53: (no value), pinhead:PINHD-1X1
- removed Q2: FA-20H, crystal:FA-20H
- removed R25, R27, R31, R32, R33, R34, R35, R36: 100, rcl:R-EU_R0402
- removed U$8: SG8002LB, sg-8002:SG8002LB
- added C23, C40: 0.47u, rcl:C-EUC0805
- added C37, C39: 3p, rcl:C-EUC0402
- added R16, R26: 3.3k, rcl:R-EU_R0402
- added R17, R22: 22k, rcl:R-EU_R0402
- added R21, R24: 2.7k, rcl:R-EU_R0402
- added U$9: SG710, SG:SG710
- C10, C13, C14, C16, C17, C20, C21, C26, C27, C28, C31, C32, C33, C34, C35, C36, C9: device rcl:C-EUC0402K -> rcl:C-EUC0402
Connections:
- net N$42 renamed DDS_OUT1B
- net N$65 renamed DDS_OUT2B
- removed net CH0_IOUT_1: R31.1
- removed net CH0_IOUT_2: R32.1
- removed net CH1_IOUT1: R25.1
- removed net CH1_IOUT2: R27.1
- removed net N$11: JP53.1, U1.FSYNC
- removed net N$13: C16.1, JP5.1, R9.2, U2.IOUT
- removed net N$14: ATMEGA328.PB6, C50.2, Q2.3
- removed net N$15: JP51.1, U1.SDATA, U2.SDATA
- removed net N$16: JP11.1, U1.SCLK, U2.SCLK
- removed net N$18: JP52.1, U2.FSYNC
- removed net N$23: C28.1, U1.DVDD
- removed net N$24: C31.1, U1.AVDD
- removed net N$64: R25.2, R36.1, U$3G$4.-IN
- removed net N$69: R27.2, R35.1, U$3G$4.+IN
- removed net N$71: C20.1, JP1.1, R7.2, U1.IOUT
- removed net N$72: C14.2, C26.1, U2.AVDD
- removed net N$73: C27.1, U2.DVDD
- removed net SDIO0: SJ2.1
- new net DDS_OUT1: C16.1, C23.1, R9.2, U2.IOUT
- new net DDS_OUT2: C20.1, C40.1, R7.2, U1.IOUT
- new net FSYNC1: U2.FSYNC
- new net FSYNC2: U1.FSYNC
- new net N$39: R24.1, U$3G$4.-IN
- new net N$91: C39.1, R22.1, R26.1, U$3G$4.+IN
- new net N$93: C40.2, R26.2
- new net SDATA: SJ2.1, U1.SDATA, U2.SDATA
- net +5V: no longer C36.1
- net 3.3V_DDS: now also C14.2, C26.1, C31.1, C36.1, U1.AVDD, U2.AVDD
- net 3.3V_MC: now also C27.1, C28.1, U1.DVDD, U2.DVDD
- net AGND: now also R21.2, R24.2
- net COS: now also C39.2, R22.2; no longer R35.2
- net GND: now also U$9.GND; no longer C43.1, C50.1, R34.2, R36.2, U$8.GND
- net N$1: now also R21.1, U$3G$1.-IN; no longer ATMEGA328.PB7, C43.2, Q2.1
- net N$76: now also C23.2, R16.2; no longer R31.2, R34.1, U$3G$1.-IN
- net N$78: now also C37.1, R16.1, R17.1; no longer R32.2, R33.1
- net N$8: now also U$9.OUT; no longer U$8.OUT
- net SCLK: now also U1.SCLK, U2.SCLK
- net SIN: now also C37.2, R17.2; no longer R33.2
- net VDD: now also U$9.VDD; no longer U$8.VDD
Other:
- moved on the sheet: U$3G$1, U$3G$4

Commit message: マイコンとオシレータ実装　あと電源周り配線
Parts:
- removed U$9: SG710, SG:SG710
- added U$8: SIT8002B, memsOsc:SIT8002B
Connections:
- removed net VDD: C32.1, U$9.VDD
- net 3.3V_MC: now also C32.1, U$8.VDD
- net GND: now also U$8.GND; no longer U$9.GND
- net N$8: now also U$8.OUT; no longer U$9.OUT
Changed lines of the file:
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@@
 <part name="U1" library="ad9834" deviceset="?AD9834" device=""/>
 <part name="U2" library="ad9834" deviceset="?AD9834" device=""/>
-<part name="VDD3" library="supply1" deviceset="VDD" device=""/>
 <part name="GND5" library="supply1" deviceset="GND" device=""/>
 <part name="GND6" library="supply1" deviceset="GND" device=""/>
@@
 <part name="R26" library="rcl" deviceset="R-EU_" device="R0402" value="3.3k"/>
 <part name="C40" library="rcl" deviceset="C-EU" device="C0805" value="0.47u"/>
-<part name="U$9" library="SG" deviceset="SG710" device=""/>
+<part name="U$8" library="memsOsc" deviceset="SIT8002B" device=""/>
 </parts>
 <sheets>
@@
 <instance part="U1" gate="G$1" x="139.7" y="40.64"/>
 <instance part="U2" gate="G$1" x="20.32" y="38.1" rot="R180"/>
-<instance part="VDD3" gate="G$1" x="81.28" y="2.54"/>
 <instance part="GND5" gate="1" x="81.28" y="-17.78"/>
 <instance part="GND6" gate="1" x="22.86" y="-5.08"/>
@@
 <instance part="C35" gate="G$1" x="170.18" y="86.36"/>
 <instance part="C36" gate="G$1" x="162.56" y="68.58"/>
-<instance part="U$9" gate="G$1" x="99.06" y="-7.62"/>
+<instance part="U$8" gate="G$1" x="99.06" y="-7.62"/>
 </instances>
 <busses>
@@
 <junction x="116.84" y="17.78"/>
 <wire x1="116.84" y1="-7.62" x2="111.76" y2="-7.62" width="0.1524" layer="91"/>
-<pinref part="U$9" gate="G$1" pin="OUT"/>
+<pinref part="U$8" gate="G$1" pin="OUT"/>
 </segment>
 </net>
@@
 <pinref part="C32" gate="G$1" pin="2"/>
 <junction x="81.28" y="-12.7"/>
-<pinref part="U$9" gate="G$1" pin="GND"/>
+<pinref part="U$8" gate="G$1" pin="GND"/>
 </segment>
 <segment>
@@
 <pinref part="C34" gate="G$1" pin="1"/>
 <pinref part="GND36" gate="1" pin="GND"/>
-</segment>
-</net>
-<net name="VDD" class="0">
-<segment>
-<wire x1="83.82" y1="-2.54" x2="81.28" y2="-2.54" width="0.1524" layer="91"/>
-<wire x1="81.28" y1="-2.54" x2="81.28" y2="-5.08" width="0.1524" layer="91"/>
-<pinref part="VDD3" gate="G$1" pin="VDD"/>
-<wire x1="81.28" y1="-2.54" x2="81.28" y2="0" width="0.1524" layer="91"/>
-<junction x="81.28" y="-2.54"/>
-<pinref part="C32" gate="G$1" pin="1"/>
-<pinref part="U$9" gate="G$1" pin="VDD"/>
 </segment>
 </net>
@@
 <label x="116.84" y="96.52" size="1.778" layer="95"/>
 </segment>
-</net>
+<segment>
+<wire x1="83.82" y1="-2.54" x2="81.28" y2="-2.54" width="0.1524" layer="91"/>
+<wire x1="81.28" y1="-2.54" x2="81.28" y2="-5.08" width="0.1524" layer="91"/>
+<wire x1="81.28" y1="-2.54" x2="81.28" y2="0" width="0.1524" layer="91"/>
+<junction x="81.28" y="-2.54"/>
+<pinref part="C32" gate="G$1" pin="1"/>
+<pinref part="U$8" gate="G$1" pin="VDD"/>
+<wire x1="81.28" y1="0" x2="73.66" y2="0" width="0.1524" layer="91"/>
+</segment>
+</net>
