File: mukumiDevice/mukumi_ad9834_wearable.sch (EAGLE design)
At the start: 136 parts, among them IC1A1 1k, IC1A1,1 1k, IC1A3'1 560, IC1B1 1k, IC1B2 1k, IC1B6,1 2k, IC2A1,1 5.1k, IC2A3 20k, IC2A3,2 20k, IC2A4 5.1k, IC2B1 20k, IC2B2 5.1k, IC2B3 20k, IC2B6,1 5.1k, IC3A2 56, IC3B1 56, IC4 TL072D, IC4A1 560, IC4A2,2 560, IC4B1 62a, IC4B2 560, IC4B6,1 560a, IC4B6,10 560a, IC4B6,11 560a, IC4B6,12 560a, IC4B6,13 560a, IC4B6,2 560a, IC4B6,3 560a, IC4B6,4 560a, IC4B6,5 560a, IC4B6,6 560a, IC4B6,7 560a, IC4B6,8 560a, IC4B6,9 560a, U1 AD9834, U2 AD9834

Commit message: DDSのAGND,GNDの間違いの修正
Connections:
- net AGND: now also R6.1, R9.1; no longer R12.2, R14.1
- net GND: now also R12.2, R14.1; no longer R6.1, R9.1
Changed lines of the file:
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@@
 <part name="GND10" library="supply1" deviceset="GND" device=""/>
 <part name="GND13" library="supply1" deviceset="GND" device=""/>
-<part name="GND19" library="supply1" deviceset="GND" device=""/>
 <part name="GND21" library="supply1" deviceset="GND" device=""/>
 <part name="GND14" library="supply1" deviceset="GND" device=""/>
-<part name="GND17" library="supply1" deviceset="GND" device=""/>
 <part name="C16" library="rcl" deviceset="C-EU" device="C0402" value="20p"/>
 <part name="C17" library="rcl" deviceset="C-EU" device="C0402" value="20p"/>
@@
 <part name="R12" library="rcl" deviceset="R-EU_" device="R0402" value="10k"/>
 <part name="R14" library="rcl" deviceset="R-EU_" device="R0402" value="10k"/>
-<part name="AGND20" library="supply1" deviceset="AGND" device=""/>
-<part name="AGND21" library="supply1" deviceset="AGND" device=""/>
 <part name="R15" library="rcl" deviceset="R-EU_" device="R0402" value="10k"/>
 <part name="GND33" library="supply1" deviceset="GND" device=""/>
@@
 <part name="C40" library="rcl" deviceset="C-EU" device="C0805" value="0.47u"/>
 <part name="U$8" library="memsOsc" deviceset="SIT8002B" device=""/>
+<part name="GND18" library="supply1" deviceset="GND" device=""/>
+<part name="GND20" library="supply1" deviceset="GND" device=""/>
+<part name="AGND11" library="supply1" deviceset="AGND" device=""/>
+<part name="AGND13" library="supply1" deviceset="AGND" device=""/>
 </parts>
 <sheets>
@@
 <instance part="GND10" gate="1" x="63.5" y="101.6" rot="R180"/>
 <instance part="GND13" gate="1" x="71.12" y="101.6" rot="R180"/>
-<instance part="GND19" gate="1" x="180.34" y="33.02"/>
 <instance part="GND21" gate="1" x="193.04" y="10.16"/>
 <instance part="GND14" gate="1" x="0" y="-20.32"/>
-<instance part="GND17" gate="1" x="7.62" y="78.74"/>
 <instance part="C16" gate="G$1" x="17.78" y="91.44"/>
 <instance part="C17" gate="G$1" x="10.16" y="-12.7"/>
@@
 <instance part="R12" gate="G$1" x="55.88" y="33.02"/>
 <instance part="R14" gate="G$1" x="66.04" y="50.8"/>
-<instance part="AGND20" gate="VR1" x="66.04" y="30.48"/>
-<instance part="AGND21" gate="VR1" x="58.42" y="48.26"/>
 <instance part="R15" gate="G$1" x="68.58" y="38.1" rot="R180"/>
 <instance part="GND33" gate="1" x="58.42" y="38.1" rot="R270"/>
@@
 <instance part="C36" gate="G$1" x="162.56" y="68.58"/>
 <instance part="U$8" gate="G$1" x="99.06" y="-7.62"/>
+<instance part="GND18" gate="1" x="66.04" y="30.48"/>
+<instance part="GND20" gate="1" x="58.42" y="48.26"/>
+<instance part="AGND11" gate="VR1" x="7.62" y="78.74"/>
+<instance part="AGND13" gate="VR1" x="180.34" y="33.02"/>
 </instances>
 <busses>
@@
 </segment>
 <segment>
-<pinref part="GND17" gate="1" pin="GND"/>
-<pinref part="R9" gate="G$1" pin="1"/>
-<wire x1="7.62" y1="81.28" x2="7.62" y2="83.82" width="0.1524" layer="91"/>
-</segment>
-<segment>
 <pinref part="R7" gate="G$1" pin="1"/>
 <pinref part="GND21" gate="1" pin="GND"/>
-</segment>
-<segment>
-<pinref part="R6" gate="G$1" pin="1"/>
-<pinref part="GND19" gate="1" pin="GND"/>
 </segment>
 <segment>
@@
 <pinref part="C34" gate="G$1" pin="1"/>
 <pinref part="GND36" gate="1" pin="GND"/>
+</segment>
+<segment>
+<pinref part="R12" gate="G$1" pin="2"/>
+<wire x1="60.96" y1="33.02" x2="66.04" y2="33.02" width="0.1524" layer="91"/>
+<pinref part="GND18" gate="1" pin="GND"/>
+</segment>
+<segment>
+<pinref part="R14" gate="G$1" pin="1"/>
+<wire x1="60.96" y1="50.8" x2="58.42" y2="50.8" width="0.1524" layer="91"/>
+<pinref part="GND20" gate="1" pin="GND"/>
 </segment>
 </net>
@@
 </segment>
 <segment>
-<pinref part="R12" gate="G$1" pin="2"/>
-<pinref part="AGND20" gate="VR1" pin="AGND"/>
-<wire x1="60.96" y1="33.02" x2="66.04" y2="33.02" width="0.1524" layer="91"/>
-</segment>
-<segment>
-<pinref part="R14" gate="G$1" pin="1"/>
-<pinref part="AGND21" gate="VR1" pin="AGND"/>
-<wire x1="60.96" y1="50.8" x2="58.42" y2="50.8" width="0.1524" layer="91"/>
-</segment>
-<segment>
 <pinref part="AGND22" gate="VR1" pin="AGND"/>
 <pinref part="C33" gate="G$1" pin="2"/>
@@
 <pinref part="C35" gate="G$1" pin="1"/>
 </segment>
-</net>
+<segment>
+<pinref part="R9" gate="G$1" pin="1"/>
+<wire x1="7.62" y1="81.28" x2="7.62" y2="83.82" width="0.1524" layer="91"/>
+<pinref part="AGND11" gate="VR1" pin="AGND"/>
+</segment>
+<segment>
+<pinref part="R6" gate="G$1" pin="1"/>
+<pinref part="AGND13" gate="VR1" pin="AGND"/>
+</segment>
+</net>
