File: mukumiDevice/mukumi_ad9834_wearable_no_power_filter.sch (EAGLE design)
At the start: 136 parts, among them IC1A1 1k, IC1A1,1 1k, IC1A3'1 560, IC1B1 1k, IC1B2 1k, IC1B6,1 2k, IC2A1,1 5.1k, IC2A3 20k, IC2A3,2 20k, IC2A4 5.1k, IC2B1 20k, IC2B2 5.1k, IC2B3 20k, IC2B6,1 5.1k, IC3A2 56, IC3B1 56, IC4 TL072D, IC4A1 560, IC4A2,2 560, IC4B1 62a, IC4B2 560, IC4B6,1 560a, IC4B6,10 560a, IC4B6,11 560a, IC4B6,12 560a, IC4B6,13 560a, IC4B6,2 560a, IC4B6,3 560a, IC4B6,4 560a, IC4B6,5 560a, IC4B6,6 560a, IC4B6,7 560a, IC4B6,8 560a, IC4B6,9 560a, U1 AD9834, U2 AD9834

Commit message: brdの一部配線、フィルタなしの構成のsch,brd追加
Parts:
- removed C1, C2, C3, C4: (no value), rcl:CPOL-EU153CLV-0807
- removed C11, C12, C15, C42: (no value), rcl:C-EUC0805
- removed U$1, U$2: D62LCB, custom parts:D62LCB
- added JP1: (no value), pinhead:PINHD-1X1
- added L1: CDRH4D18, inductor-sumida:CDRH4D18
- added R3: 1k, rcl:R-EU_R0402
Connections:
- removed net +REG: C11.1, C4.+, JP2.2, U$1.P$1
- removed net -REG: C15.1, C2.+, JP2.4, U$2.P$1
- removed net CS: ATMEGA328.PD6
- removed net IO_UPDATE: ATMEGA328.PD7
- removed net MASTER_RESET: ATMEGA328.PD5
- new net ANALOGSWITCH: ATMEGA328.PD5, JP1.1, R3.2
- new net N$11: R3.1, U$8.OE
- net +5V: now also JP2.2; no longer C1.+, C12.1, U$1.P$2
- net -5V: now also JP2.4; no longer C3.+, C42.1, U$2.P$2
- net AGND: now also C18.2, C19.2, L1.1, R6.1, R7.1, R8.1, R9.1, U$5.GND; no longer R12.2, R14.1
- net GND: now also L1.2, R12.2, R14.1; no longer C1.-, C11.2, C12.2, C15.2, C18.2, C19.2, C2.-, C3.-, C4.-, C42.2, R6.1, R7.1, R8.1, R9.1, U$5.GND
Other:
- moved on the sheet: R14, R15
