File: mukumiDevice/mukumi_ad9834_wearable_no_power_filter.sch (EAGLE design)
At the start: 129 parts, among them IC1A1 1k, IC1A1,1 1k, IC1A3'1 560, IC1B1 1k, IC1B2 1k, IC1B6,1 2k, IC2A1,1 5.1k, IC2A3 20k, IC2A3,2 20k, IC2A4 5.1k, IC2B1 20k, IC2B2 5.1k, IC2B3 20k, IC2B6,1 5.1k, IC3A2 56, IC3B1 56, IC4 TL072D, IC4A1 560, IC4A2,2 560, IC4B1 62a, IC4B2 560, IC4B6,1 560a, IC4B6,10 560a, IC4B6,11 560a, IC4B6,12 560a, IC4B6,13 560a, IC4B6,2 560a, IC4B6,3 560a, IC4B6,4 560a, IC4B6,5 560a, IC4B6,6 560a, IC4B6,7 560a, IC4B6,8 560a, IC4B6,9 560a, U1 AD9834, U2 AD9834

Commit message: Revert "agnd,dgndのインダクタによる接続"
This reverts commit 8ebf4f6ca6ba426166226e421df2150118e3df71.
Parts:
- L1: value CB2016 -> CDRH4D18; device inductor-yuden:CB2016 -> inductor-sumida:CDRH4D18
Changed lines of the file:
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@@
 <part name="AGND18" library="supply1" deviceset="AGND" device=""/>
 <part name="GND11" library="supply1" deviceset="GND" device=""/>
+<part name="L1" library="inductor-sumida" deviceset="CDRH4D18" device=""/>
 <part name="P+4" library="supply1" deviceset="+5V" device=""/>
 <part name="P-11" library="supply1" deviceset="-5V" device=""/>
-<part name="L1" library="inductor-yuden" deviceset="CB2016" device=""/>
 </parts>
 <sheets>
@@
 <instance part="AGND18" gate="VR1" x="114.3" y="50.8"/>
 <instance part="GND11" gate="1" x="129.54" y="50.8"/>
+<instance part="L1" gate="G$1" x="121.92" y="53.34"/>
 <instance part="P+4" gate="1" x="30.48" y="50.8" rot="R270"/>
 <instance part="P-11" gate="1" x="30.48" y="55.88" rot="R90"/>
-<instance part="L1" gate="G$1" x="121.92" y="53.34"/>
 </instances>
 <busses>
@@
 </segment>
 <segment>
+<pinref part="L1" gate="G$1" pin="2"/>
 <pinref part="GND11" gate="1" pin="GND"/>
 <wire x1="127" y1="53.34" x2="129.54" y2="53.34" width="0.1524" layer="91"/>
-<pinref part="L1" gate="G$1" pin="2"/>
 </segment>
 </net>
@@
 </segment>
 <segment>
+<pinref part="L1" gate="G$1" pin="1"/>
 <pinref part="AGND18" gate="VR1" pin="AGND"/>
 <wire x1="116.84" y1="53.34" x2="114.3" y2="53.34" width="0.1524" layer="91"/>
-<pinref part="L1" gate="G$1" pin="1"/>
-</segment>
-</net>
+</segment>
+</net>
