File: mukumiDevice/mukumi_ad9834_wearable_no_power_filter.sch (EAGLE design)
At the start: 131 parts, among them IC1A1 1k, IC1A1,1 1k, IC1A3'1 560, IC1B1 1k, IC1B2 1k, IC1B6,1 2k, IC2A1,1 5.1k, IC2A3 20k, IC2A3,2 20k, IC2A4 5.1k, IC2B1 20k, IC2B2 5.1k, IC2B3 20k, IC2B6,1 5.1k, IC3A2 56, IC3B1 56, IC4 TL072D, IC4A1 560, IC4A2,2 560, IC4B1 62a, IC4B2 560, IC4B6,1 560a, IC4B6,10 560a, IC4B6,11 560a, IC4B6,12 560a, IC4B6,13 560a, IC4B6,2 560a, IC4B6,3 560a, IC4B6,4 560a, IC4B6,5 560a, IC4B6,6 560a, IC4B6,7 560a, IC4B6,8 560a, IC4B6,9 560a, U1 AD9834, U2 AD9834

Commit message: bNAMEの整理と部品名の整理
Parts:
- renumbered AD633_1 to IC1, AD633_2 to IC2, AD633_3 to IC3, C,IC2A1 to C50, C,IC2A10 to C42, C,IC2A11 to C54, C,IC2A12 to C53, C,IC2A13 to C49, C,IC2A14 to C55, C,IC2A15 to C43, C,IC2A16 to C44, C,IC2A17 to C45, C,IC2A18 to C46, C,IC2A2 to C11, C,IC2A3 to C2, C,IC2A4 to C22, C,IC2A5 to C41, C,IC2A6 to C48, C,IC2A7 to C1, C,IC2A8 to C12, C,IC2A9 to C38, C,IC4A1,1 to C4, CIC2B1 to C3, IC1A1 to R20, IC1A1,1 to R23, IC1A3'1 to R13, IC1B1 to R25, IC1B2 to R27, IC1B6,1 to R28, IC2A1,1 to R34, IC2A3 to R33, IC2A3,2 to R35, IC2A4 to R36, IC2B1 to R29, IC2B2 to R31, IC2B3 to R32, IC2B6,1 to R30, IC3A2 to R38, IC3B1 to R37, IC4A1 to R39, IC4A2,2 to R40, IC4B1 to R42, IC4B2 to R41, IC4B6,1 to R43, IC4B6,10 to R45, IC4B6,11 to R49, IC4B6,12 to R52, IC4B6,13 to R53, IC4B6,2 to R46, IC4B6,3 to R47, IC4B6,4 to R50, IC4B6,5 to R51, IC4B6,6 to R54, IC4B6,7 to R55, IC4B6,8 to R44, IC4B6,9 to R48, L2 to L1, U$1 to IC9, U$10 to IC7, U$11 to IC5, U$2 to IC10, U$3 to IC6, U$4 to VR1, U$7 to IC8, U$8 to IC13, U1 to IC12, U2 to IC11
