File: mukumiDevice/mukumi_ad9834_wearable_no_power_filter_re_line.brd (EAGLE design)
At the start: 54 x 41.7 mm, 131 parts, among them IC1 AD835, IC10 NJM2884, IC11 AD9834, IC12 AD9834, IC13 SIT8002B, IC2 AD835, IC3 AD835, IC4 TL072D, IC5 NJM074V, IC6 NJM074V, IC7 NJM074V, IC8 NJM074V, IC9 NJM2884

Commit message: パターンを太くしたバージョン追加、ベタパターン追加、ｐ板提供部品に合わせたコンデンサ部品サイズの変更、DDSのfsyncがつながっていなかったのを修正、テスト、調整用スルーホール追加
Parts:
- added D1, D2, D3, D4: (no value), microbuilder:SOD-523
- added SJ3: (no value), jumper:SJ
- C29, C30, C5, C6, C7, C8: value (none) -> 0.47u
- R1: value (none) -> 10k
- R45: value 560a -> 100k
- R49: value 560a -> 47k
- moved R3 3.55 mm to (8.16, 16.6), turned to 180 degrees
- moved C50 1.70 mm to (25.8, 27.0)
- moved C7 0.51 mm to (30.5, 4.72)
- moved L1 0.43 mm to (13.1, 34.0), turned to 270 degrees
- moved C40 0.30 mm to (20.2, 27.5)
Connections:
- removed net N$38: IC12.12
- new net SIG_: IC1.8, IC2.8, SJ3.2
- net 3.3V_DDS: now also ATMEGA328.18
- net 3.3V_MC: now also D2.K, D4.K; no longer ATMEGA328.18
- net AGND: now also ATMEGA328.21, D1.A, D3.A
- net ANALOGSWITCH: now also ATMEGA328.11; no longer ATMEGA328.9
- net FSYNC1: now also ATMEGA328.9
- net FSYNC2: now also ATMEGA328.10
- net GND: now also IC11.12, IC12.12; no longer ATMEGA328.21
- net SIG: now also SJ3.1; no longer IC1.8, IC2.8
- net SIG*COS: now also D3.K, D4.A
- net SIG*SIN: now also D1.K, D2.A
Routing:
- net AGND: track 321.1 -> 357.8 mm, vias 21 -> 22
- net 3.3V_DDS: track 42.4 -> 75.8 mm, vias 2 -> 3
- net SIG_: track 0.00 -> 24.2 mm, vias 0 -> 1
- net SIG: track 31.6 -> 8.77 mm
- net FSYNC2: track 0.00 -> 22.4 mm, vias 0 -> 2
- net -5V: track 118.6 -> 100.4 mm
- net 3.3V_MC: track 81.1 -> 98.6 mm
- net FSYNC1: track 0.00 -> 15.8 mm, vias 0 -> 1
- net SIG*COS: track 18.9 -> 28.7 mm, vias 2 -> 3
- net N$45: track 15.0 -> 6.70 mm
- net GND: track 147.2 -> 139.6 mm
- net N$44: track 15.0 -> 20.0 mm
- net +5V: track 110.7 -> 115.0 mm
- net SIG*SIN: track 20.7 -> 24.9 mm, vias 2 -> 3
- net N$11: track 10.0 -> 7.74 mm
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