File: mukumiDevice/mukumi_ad9834_wearable_add_solid_pattern.sch (EAGLE design)
At the start: 131 parts, among them IC4 TL072D, U1 AD9834, U2 AD9834

Commit message: パターンを太くしたバージョン追加、ベタパターン追加、ｐ板提供部品に合わせたコンデンサ部品サイズの変更、DDSのfsyncがつながっていなかったのを修正、テスト、調整用スルーホール追加
Parts:
- added D1, D2, D3, D4: (no value), microbuilder:DIODESOD-523
- added SJ3: (no value), jumper:SJ
- C18, C19, C24, C25: device rcl:C-EUC0402 -> rcl:C-EUC0603
- C29, C30, C5, C6, C7, C8: value (none) -> 0.47u
- R1: value (none) -> 10k
- R45: value 560a -> 100k
- R49: value 560a -> 47k
- renumbered AD633_1 to IC1, AD633_2 to IC2, AD633_3 to IC3, U$1 to IC9, U$10 to IC7, U$11 to IC5, U$2 to IC10, U$3 to IC6, U$7 to IC8, U$8 to IC13, U1 to IC12, U2 to IC11
Connections:
- removed net N$38: IC12.SLEEP
- new net SIG_: IC1.X1, IC2.X1, SJ3.2
- net 3.3V_DDS: now also ATMEGA328.AVCC
- net 3.3V_MC: now also D2.C, D4.C; no longer ATMEGA328.AVCC
- net AGND: now also ATMEGA328.GND, D1.A, D3.A
- net ANALOGSWITCH: now also ATMEGA328.PD7; no longer ATMEGA328.PD5
- net FSYNC1: now also ATMEGA328.PD5
- net FSYNC2: now also ATMEGA328.PD6
- net GND: now also IC11.SLEEP, IC12.SLEEP; no longer ATMEGA328.GND
- net SIG: now also SJ3.1; no longer IC1.X1, IC2.X1
- net SIG*COS: now also D3.C, D4.A
- net SIG*SIN: now also D1.C, D2.A

Commit message: 電源パターンの調整、SIN,COSデバッグ用ビアの追加、インダクタの変更
ガーバーファイル追加
Parts:
- L1: value CB2016 -> CDRH4D18; device inductor-yuden:CB2016 -> inductor-sumida:CDRH4D18
Changed lines of the file:
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@@
 <part name="P+4" library="supply1" deviceset="+5V" device=""/>
 <part name="P-11" library="supply1" deviceset="-5V" device=""/>
-<part name="L1" library="inductor-yuden" deviceset="CB2016" device=""/>
+<part name="L1" library="inductor-sumida" deviceset="CDRH4D18" device=""/>
 <part name="IC9" library="torex" deviceset="NJM2884" device=""/>
 <part name="IC10" library="torex" deviceset="NJM2884" device=""/>
