File: mukumiDevice/mukumi_ad9834_wearable_add_solid_pattern.sch (EAGLE design)
At the start: 141 parts, among them IC1 AD835, IC10 NJM2884, IC11 AD9834, IC12 AD9834, IC13 SIT8002B, IC2 AD835, IC3 AD835, IC4 TL072D, IC5 NJM074V, IC6 NJM074V, IC7 NJM074V, IC8 NJM074V, IC9 NJM2884

Commit message: 負電圧の信号を取るため、atmega328のPWM(analogWrite)とRCローパスを用いてVCC/2を生成し、それを抵抗(1.8kのやつ）で加算してからAD変換ポートにつなぐ
Parts:
- R20: value 1k -> 680
- R23: value 1k -> 360
- R28: value 2k -> 1k
- R45: value 100k -> 11k
- R49: value 47k -> 11k
Changed lines of the file:
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@@
 <part name="R34" library="rcl" deviceset="R-EU_" device="R0402" value="5.1k"/>
 <part name="R36" library="rcl" deviceset="R-EU_" device="R0402" value="5.1k"/>
-<part name="R23" library="rcl" library_urn="urn:adsk.eagle:library:334" deviceset="R-EU_" device="R0402" value="1k"/>
-<part name="R20" library="rcl" library_urn="urn:adsk.eagle:library:334" deviceset="R-EU_" device="R0402" value="1k"/>
+<part name="R23" library="rcl" library_urn="urn:adsk.eagle:library:334" deviceset="R-EU_" device="R0402" value="360"/>
+<part name="R20" library="rcl" library_urn="urn:adsk.eagle:library:334" deviceset="R-EU_" device="R0402" value="680"/>
 <part name="R35" library="rcl" deviceset="R-EU_" device="R0402" value="20k"/>
 <part name="GND15" library="supply1" deviceset="AGND" device=""/>
@@
 <part name="C3" library="rcl" deviceset="C-EU" device="C2012" value="4.7u"/>
 <part name="GND63" library="supply1" deviceset="AGND" device=""/>
-<part name="R28" library="rcl" library_urn="urn:adsk.eagle:library:334" deviceset="R-EU_" device="R0402" value="2k"/>
+<part name="R28" library="rcl" library_urn="urn:adsk.eagle:library:334" deviceset="R-EU_" device="R0402" value="1k"/>
 <part name="R25" library="rcl" library_urn="urn:adsk.eagle:library:334" deviceset="R-EU_" device="R0402" value="1k"/>
 <part name="R27" library="rcl" deviceset="R-EU_" device="R0402" value="1k"/>
@@
 <part name="R44" library="rcl" deviceset="R-EU_" device="R0402" value="560a"/>
 <part name="R48" library="rcl" deviceset="R-EU_" device="R0402" value="560a"/>
-<part name="R45" library="rcl" deviceset="R-EU_" device="R0402" value="100k"/>
-<part name="R49" library="rcl" deviceset="R-EU_" device="R0402" value="47k"/>
+<part name="R45" library="rcl" deviceset="R-EU_" device="R0402" value="11k"/>
+<part name="R49" library="rcl" deviceset="R-EU_" device="R0402" value="11k"/>
 <part name="IC3" library="linear" deviceset="AD835" device=""/>
 <part name="P+13" library="supply1" deviceset="+5V" device=""/>

Commit message: 装置回路図に加算回路の追加
Parts:
- added IC14: NJM074V, linear:NJM074V
- added R59, R60, R61, R62, R63, R64, R65, R66, R67, R68, R69, R70, R71, R72: 560a, rcl:R-EU_R0402
Connections:
- new net AOUT1: ATMEGA328.PC0, IC14G$3.OUT, R70.2
- new net AOUT2: ATMEGA328.PC1, IC14G$2.OUT, R63.2
- new net N$31: IC14G$1.-IN, R59.2, R60.2, R61.1
- new net N$32: IC14G$2.-IN, R62.2, R63.1
- new net N$37: IC14G$1.OUT, R61.2, R62.1
- new net N$38: IC14G$4.-IN, R66.2, R67.2, R68.1
- new net N$39: IC14G$3.-IN, R69.2, R70.1
- new net N$42: IC14G$4.OUT, R68.2, R69.1
- new net VCC: R64.2
- new net VCC/2: R59.1, R64.1, R65.2
- new net VCC/22: R66.1, R71.1, R72.2
- new net VCC2: R71.2
- net +5V: now also IC14G$1.V-
- net -5V: now also IC14G$1.V+
- net AGND: now also IC14G$1.+IN, IC14G$2.+IN, IC14G$3.+IN, IC14G$4.+IN, R65.1, R72.1
- net SIG*COS: now also R60.1; no longer ATMEGA328.PC1
- net SIG*SIN: now also R67.1; no longer ATMEGA328.PC0
Other:
- moved on the sheet: C43, C44, C45, C46, C48, C49, C50, C53, C54, C55

Commit message: 回路図のセラミックコンデンサから電解コンデンサへの置換、加算回路のvcc/2をdds電源からの生成へ変更、基板サイズ拡大
Parts:
- removed C29, C30, C5, C6, C7, C8: 0.47u, rcl:C-EUC0805
- added C15, C47, C56, C57, C58, C59: (no value), rcl:CPOL-EUB
- C2, C3: value 4.7u -> 0.47u; device rcl:C-EUC2012 -> rcl:CPOL-EUB
- C23, C40: value 0.47u -> 4.7u; device rcl:C-EUC0805 -> rcl:CPOL-EUB
- C4: device rcl:C-EUC2012 -> rcl:CPOL-EUB
Connections:
- removed net N$76: C23.2, R16.2
- removed net N$93: C40.2, R26.2
- removed net VCC: R64.2
- removed net VCC2: R71.2
- new net N$45: C4.-, R26.2
- new net N$64: C3.-, R16.2
- net 3.3V_DDS: now also R64.2, R71.2
- net A1: now also C40.+; no longer C3.1
- net AGND: now also C15.-, C56.-, C58.-; no longer C30.1, C6.1, C7.1
- net DDS_OUT1: now also C3.+; no longer C23.1
- net DDS_OUT2: now also C4.+; no longer C40.1
- net N$19: now also C15.+; no longer C30.2
- net N$2: now also C56.+; no longer C6.2
- net N$3: now also C58.+; no longer C7.2
- net N$4: now also C57.+; no longer C5.1
- net N$41: now also C23.-; no longer C2.2
- net N$46: now also C40.-; no longer C3.2
- net N$54: now also C2.+; no longer C4.1
- net N$55: now also C2.-; no longer C4.2
- net N$56: now also C23.+; no longer C2.1
- net N$6: now also C59.+; no longer C8.2
- net N$63: now also C47.+; no longer C29.1
- net SIG*COS: now also C57.-; no longer C5.2
- net SIG*SIN: now also C59.-; no longer C8.1
- net SIN*SIN: now also C47.-; no longer C29.2

Commit message: brdに加算回路追加
Parts:
- removed C15, C47: (no value), rcl:CPOL-EUB
- removed IC3: AD835, linear:AD835
- removed IC4: TL072D, linear:TL072D
- removed R52, R53, R54, R55, R58: 560a, rcl:R-EU_R0402
Connections:
- removed net N$12: IC4A.OUT, R53.2, R54.1
- removed net N$16: IC4A.+IN, R58.2
- removed net N$19: C15.+, IC4B.+IN, R55.2
- removed net N$5: IC3.W, R58.1
- removed net N$63: C47.+, R54.2, R55.1
- removed net N$70: IC4A.-IN, R52.2, R53.1
- net +5V: no longer IC3.VP, IC4P.V+
- net -5V: no longer IC3.VN, IC4P.V-
- net AGND: no longer C15.-, IC3.X1, IC3.Y2, IC3.Z, R52.1
- net AOUT1: now also D1.C, D2.A
- net AOUT2: now also D3.C, D4.A
- net SIG*COS: no longer D3.C, D4.A
- net SIG*SIN: no longer D1.C, D2.A
- net SIN*SIN: no longer C47.-, IC4B.-IN, IC4B.OUT
- net SIN_: no longer IC3.X2, IC3.Y1
Other:
- moved on the sheet: D1, D2, D3, D4
