File: mukumiDevice/mukumi_ad9834_wearable_add_solid_pattern.brd (EAGLE design)
At the start: 49.2 x 41.7 mm, 156 parts, among them IC1 AD835, IC10 NJM2884, IC11 AD9834, IC12 AD9834, IC13 SIT8002B, IC14 NJM074V, IC2 AD835, IC3 AD835, IC4 TL072D, IC5 NJM074V, IC6 NJM074V, IC7 NJM074V, IC8 NJM074V, IC9 NJM2884

Commit message: 回路図のセラミックコンデンサから電解コンデンサへの置換、加算回路のvcc/2をdds電源からの生成へ変更、基板サイズ拡大
Parts:
- removed C29, C30, C5, C6, C7, C8: 0.47u, rcl:C0805
- added C15, C47, C56, C57, C58, C59: (no value), rcl:PANASONIC_B
- C2, C3: value 4.7u -> 0.47u; device rcl:C2012 -> rcl:PANASONIC_B
- C23, C40: value 0.47u -> 4.7u; device rcl:C0805 -> rcl:PANASONIC_B
- C4: device rcl:C2012 -> rcl:PANASONIC_B
- moved C23 45.5 mm to (58.5, 42.4), turned to 0 degrees
- moved C40 42.4 mm to (58.5, 36.4), flipped to the top, turned to 0 degrees
- moved C3 40.1 mm to (58.5, 54.4), flipped to the top
- moved IC14 37.3 mm to (-17.2, 25.6)
- moved R59 37.3 mm to (-11.3, 27.8)
- moved R60 37.3 mm to (-5.90, 27.8)
- moved R61 37.3 mm to (-20.0, 18.8)
- moved R62 37.3 mm to (-14.6, 18.8)
- moved R63 37.3 mm to (-9.20, 18.8)
- moved R64 37.3 mm to (-20.0, 13.9)
- moved R65 37.3 mm to (-14.6, 13.9)
- moved R66 37.3 mm to (-9.20, 13.9)
- moved R67 37.3 mm to (-20.0, 9.00)
- moved R68 37.3 mm to (-14.6, 9.00)
- moved R69 37.3 mm to (-9.20, 9.00)
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Connections:
- removed net N$76: C23.2, R16.2
- removed net N$93: C40.2, R26.2
- removed net VCC: R64.2
- removed net VCC2: R71.2
- new net N$45: C4.-, R26.2
- new net N$64: C3.-, R16.2
- net 3.3V_DDS: now also R64.2, R71.2
- net A1: now also C40.+; no longer C3.1
- net AGND: now also C15.-, C56.-, C58.-; no longer C30.1, C6.1, C7.1
- net DDS_OUT1: now also C3.+; no longer C23.1
- net DDS_OUT2: now also C4.+; no longer C40.1
- net N$19: now also C15.+; no longer C30.2
- net N$2: now also C56.+; no longer C6.2
- net N$3: now also C58.+; no longer C7.2
- net N$4: now also C57.+; no longer C5.1
- net N$41: now also C23.-; no longer C2.2
- net N$46: now also C40.-; no longer C3.2
- net N$54: now also C2.+; no longer C4.1
- net N$55: now also C2.-; no longer C4.2
- net N$56: now also C23.+; no longer C2.1
- net N$6: now also C59.+; no longer C8.2
- net N$63: now also C47.+; no longer C29.1
- net SIG*COS: now also C57.-; no longer C5.2
- net SIG*SIN: now also C59.-; no longer C8.1
- net SIN*SIN: now also C47.-; no longer C29.2
Routing:
- net AGND: track 367.9 -> 364.6 mm
- net N$55: track 7.75 -> 5.13 mm
- net N$76: track 2.60 -> 0.00 mm
- net SIG*COS: track 20.2 -> 17.7 mm
- net SIN*SIN: track 40.0 -> 37.6 mm
- net N$19: track 3.52 -> 1.73 mm
- net N$46: track 2.12 -> 0.33 mm
- net N$63: track 15.2 -> 13.6 mm
- net N$93: track 1.66 -> 0.00 mm
- net N$54: track 4.47 -> 3.14 mm
- net SIG*SIN: track 21.8 -> 20.6 mm
- net N$41: track 1.83 -> 0.83 mm
- net DDS_OUT1: track 6.54 -> 5.77 mm
- net N$6: track 7.56 -> 7.02 mm
Other:
- board size 49.2 x 41.7 mm -> 49.2 x 49.6 mm

Commit message: brdに加算回路追加
Parts:
- removed C15, C47: (no value), rcl:PANASONIC_B
- removed IC3: AD835, linear:SO08
- removed IC4: TL072D, linear:SO08
- removed R52, R53, R54, R55, R58: 560a, rcl:R0402
- moved R70 66.0 mm to (45.4, 12.7), flipped to the bottom
- moved R67 62.3 mm to (42.2, 6.10), flipped to the bottom
- moved R71 61.4 mm to (46.6, 9.40), flipped to the bottom, turned to 180 degrees
- moved IC14 59.4 mm to (40.3, 10.6), flipped to the bottom, turned to 90 degrees
- moved R61 59.3 mm to (38.2, 7.30), flipped to the bottom
- moved R69 57.3 mm to (48.0, 12.7), flipped to the bottom, turned to 90 degrees
- moved R68 57.2 mm to (42.6, 7.30), flipped to the bottom, turned to 180 degrees
- moved R72 56.2 mm to (46.6, 10.6), flipped to the bottom
- moved R64 54.1 mm to (34.0, 10.3), flipped to the bottom, turned to 90 degrees
- moved R66 53.8 mm to (44.4, 9.80), flipped to the bottom, turned to 270 degrees
- moved R59 50.9 mm to (36.3, 9.80), flipped to the bottom, turned to 270 degrees
- moved R65 49.8 mm to (35.1, 10.3), flipped to the bottom, turned to 270 degrees
- moved R62 47.2 mm to (31.7, 9.80), flipped to the bottom, turned to 90 degrees
- moved R63 47.0 mm to (37.5, 13.9), flipped to the bottom, turned to 270 degrees
- moved R60 41.2 mm to (32.6, 13.0), flipped to the bottom, turned to 270 degrees
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Connections:
- removed net N$12: IC4.1, R53.2, R54.1
- removed net N$16: IC4.3, R58.2
- removed net N$19: C15.+, IC4.5, R55.2
- removed net N$5: IC3.5, R58.1
- removed net N$63: C47.+, R54.2, R55.1
- removed net N$70: IC4.2, R52.2, R53.1
- net +5V: no longer IC3.6, IC4.8
- net -5V: no longer IC3.3, IC4.4
- net AGND: no longer C15.-, IC3.2, IC3.4, IC3.8, R52.1
- net AOUT1: now also D1.K, D2.A
- net AOUT2: now also D3.K, D4.A
- net SIG*COS: no longer D3.K, D4.A
- net SIG*SIN: no longer D1.K, D2.A
- net SIN*SIN: no longer C47.-, IC4.6, IC4.7
- net SIN_: no longer IC3.1, IC3.7
Routing:
- net 3.3V_DDS: track 65.5 -> 123.1 mm, vias 3 -> 5
- net SIN*SIN: track 37.6 -> 0.00 mm, vias 1 -> 0
- net AOUT1: track 0.00 -> 29.3 mm
- net SIG*SIN: track 20.6 -> 43.7 mm
- net AOUT2: track 0.00 -> 22.7 mm
- net N$32: track 0.00 -> 16.4 mm
- net AGND: track 364.6 -> 380.5 mm
- net SIN_: track 30.0 -> 15.0 mm
- net SIG*COS: track 17.7 -> 31.3 mm, vias 3 -> 4
- net N$63: track 13.6 -> 0.00 mm, vias 2 -> 0
- net N$6: track 7.02 -> 19.2 mm, vias 0 -> 1
- net N$31: track 0.00 -> 11.6 mm
- net N$42: track 0.00 -> 11.3 mm
- net GND: track 186.6 -> 196.4 mm, vias 5 -> 4
- net N$12: track 9.56 -> 0.00 mm
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
Commit message: brdのacカップリングコンデンサを電解コンデンサへの置換
Parts:
- moved C3 51.5 mm to (21.0, 19.1), turned to 90 degrees
- moved C4 46.2 mm to (17.5, 27.1), turned to 270 degrees
- moved C2 38.4 mm to (45.3, 24.3), turned to 270 degrees
- moved C40 27.7 mm to (34.4, 22.8)
- moved C23 26.3 mm to (34.8, 30.9), turned to 270 degrees
- moved R32 2.50 mm to (36.5, 26.5)
- moved R57 1.90 mm to (34.1, 8.70)
- moved R16 1.00 mm to (16.8, 20.9)
- moved R30 0.91 mm to (30.6, 22.5), turned to 270 degrees
- moved R31 0.62 mm to (33.4, 25.8), turned to 180 degrees
- moved R70 0.61 mm to (45.5, 13.3)
- moved R10 0.41 mm to (17.9, 18.1)
- moved C39 0.40 mm to (16.7, 33.9)
- moved R26 0.22 mm to (17.6, 30.6)
- moved C21 0.20 mm to (14.5, 31.5)
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Routing:
- net AOUT2: track 22.7 -> 39.4 mm, vias 0 -> 1
- net AOUT1: track 29.3 -> 45.4 mm, vias 0 -> 1
- net DDS_OUT1: track 5.77 -> 14.0 mm, vias 0 -> 1
- net N$54: track 3.14 -> 11.0 mm, vias 0 -> 1
- net N$64: track 0.00 -> 7.09 mm, vias 0 -> 1
- net N$4: track 15.6 -> 11.2 mm
- net N$55: track 5.13 -> 9.58 mm
- net N$58: track 10.7 -> 6.77 mm
- net N$32: track 16.4 -> 20.3 mm
- net N$41: track 0.83 -> 4.57 mm, vias 0 -> 1
- net N$46: track 0.33 -> 3.78 mm
- net SIG: track 9.09 -> 11.9 mm
- net AGND: track 380.5 -> 378.0 mm, vias 25 -> 26
- net N$91: track 9.39 -> 11.7 mm
- net A1: track 3.03 -> 5.28 mm
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