File: mukumiDevice/utility.brd (EAGLE design)
At the start: 51 x 43.6 mm, 12 parts

Commit message: P板からの指摘点を修正、ad633用ユーティリティ基板の作成
Parts:
- moved JP8 0.36 mm to (27.7, 40.7)
- moved JP1 0.32 mm to (41.2, 40.7)
- moved JP2 0.22 mm to (15.0, 4.87)
Routing:
- added copper zone on layer 16, net N$6
Changed lines of the file:
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@@
 <elements>
 <element name="CURRENT_OUT" library="audiojack" package="3.5MM" value="STEREO3.5MM" x="48.49" y="8.18" rot="MR0"/>
-<element name="JP1" library="pinhead" package="1X05" value="" x="41.27" y="40.97" rot="R180"/>
-<element name="JP2" library="pinhead" package="1X06" value="" x="15.095" y="4.67" rot="R180"/>
+<element name="JP1" library="pinhead" package="1X05" value="" x="41.17" y="40.67" rot="R180"/>
+<element name="JP2" library="pinhead" package="1X06" value="" x="14.995" y="4.87" rot="R180"/>
 <element name="JP7" library="pinhead" package="1X06" value="" x="10.65" y="40.98"/>
-<element name="JP8" library="pinhead" package="1X04" value="" x="27.87" y="41.02" rot="R180"/>
+<element name="JP8" library="pinhead" package="1X04" value="" x="27.67" y="40.72" rot="R180"/>
 <element name="JP9" library="pinhead" package="1X01" value="" x="22.45" y="8.46" rot="MR0"/>
 <element name="MESURE_VOL" library="audiojack" package="3.5MM" value="STEREO3.5MM" x="48.57" y="27.22" rot="MR0"/>
@@
 <wire x1="48.47" y1="8.841" x2="48.57" y2="27.22" width="1.27" layer="16"/>
 <wire x1="48.49" y1="9.01" x2="48.49" y2="8.18" width="1.27" layer="16"/>
-<wire x1="41.27" y1="40.97" x2="41.17" y2="27.83355" width="1.27" layer="16"/>
+<wire x1="41.17" y1="40.67" x2="41.17" y2="27.83355" width="1.27" layer="16"/>
 <wire x1="43.1074" y1="26.69615" x2="41.17" y2="27.83355" width="1.27" layer="16"/>
 <wire x1="43.1074" y1="19.5449" x2="43.1074" y2="26.69615" width="1.27" layer="16"/>
@@
 <wire x1="41.0526" y1="14.7" x2="42.5526" y2="17.3901" width="1.016" layer="16"/>
 <wire x1="42.5526" y1="17.3901" x2="43.1074" y2="19.5449" width="1.016" layer="16"/>
-<wire x1="41.27" y1="40.97" x2="41.27" y2="40.93" width="1.27" layer="16"/>
+<wire x1="41.17" y1="40.67" x2="41.27" y2="40.93" width="1.27" layer="16"/>
 <wire x1="41.27" y1="40.93" x2="41.3" y2="40.9" width="1.27" layer="16"/>
 <wire x1="41.3" y1="40.9" x2="41.3" y2="40.94" width="1.27" layer="16"/>
-<wire x1="41.3" y1="40.94" x2="41.27" y2="40.97" width="1.27" layer="16"/>
+<wire x1="41.3" y1="40.94" x2="41.17" y2="40.67" width="1.27" layer="16"/>
 </signal>
 <signal name="N$2">
 <contactref element="CURRENT_OUT" pad="P$4"/>
 <contactref element="JP1" pad="1"/>
-<wire x1="46.7326" y1="40.5874" x2="46.35" y2="40.97" width="1.27" layer="16"/>
+<wire x1="46.7326" y1="40.5874" x2="46.25" y2="40.67" width="1.27" layer="16"/>
 <wire x1="46.7326" y1="31.1" x2="46.7326" y2="40.5874" width="1.27" layer="16"/>
 <wire x1="43.29" y1="12.78" x2="43.29" y2="12.9425" width="1.27" layer="16"/>
@@
 <wire x1="37.9" y1="18.46725625" x2="37.9" y2="18" width="1.27" layer="16"/>
 <wire x1="37.1092125" y1="19.836359375" x2="37.9" y2="18.46725625" width="1.27" layer="16"/>
-<wire x1="36.19" y1="40.97" x2="36.19" y2="33.80454375" width="1.27" layer="16"/>
+<wire x1="36.09" y1="40.67" x2="36.19" y2="33.80454375" width="1.27" layer="16"/>
 <wire x1="36.19" y1="33.80454375" x2="37.7824" y2="32.21214375" width="1.27" layer="16"/>
 <wire x1="37.7824" y1="32.21214375" x2="37.7824" y2="29.0824" width="1.27" layer="16"/>
@@
 <contactref element="MESURE_VOL" pad="P$4"/>
 <contactref element="JP1" pad="2"/>
-<wire x1="43.81" y1="40.97" x2="43.81" y2="32.26" width="1.27" layer="16"/>
+<wire x1="43.71" y1="40.67" x2="43.81" y2="32.26" width="1.27" layer="16"/>
 <wire x1="43.81" y1="32.26" x2="43.37" y2="31.82" width="1.27" layer="16"/>
 </signal>
@@
 <wire x1="38.67" y1="22.03" x2="37.2" y2="23.5" width="1.27" layer="16"/>
 <wire x1="37.2" y1="25.6" x2="37.2" y2="23.5" width="1.27" layer="16"/>
-<wire x1="38.73" y1="40.97" x2="38.73" y2="34.38158125" width="1.27" layer="16"/>
+<wire x1="38.63" y1="40.67" x2="38.73" y2="34.38158125" width="1.27" layer="16"/>
 <wire x1="38.73" y1="34.38158125" x2="39.5224" y2="33.48918125" width="1.27" layer="16"/>
 <wire x1="39.5224" y1="33.48918125" x2="39.5224" y2="28.2224" width="1.27" layer="16"/>
@@
 <contactref element="R2" pad="2"/>
 <contactref element="CURRENT_OUT" pad="P$5"/>
-<wire x1="35.57" y1="31.52" x2="35.87" y2="30.3368125" width="1.27" layer="16"/>
-<wire x1="35.87" y1="30.3368125" x2="32.16659375" y2="26.63340625" width="1.27" layer="16"/>
+<wire x1="35.57" y1="31.52" x2="35.57" y2="29.3368125" width="1.27" layer="16"/>
+<wire x1="35.57" y1="29.3368125" x2="32.16659375" y2="26.23340625" width="1.27" layer="16"/>
 <wire x1="32.64" y1="18.54" x2="35.93" y2="18.54" width="1.27" layer="16"/>
 <wire x1="32.16659375" y1="18.06659375" x2="32.64" y2="18.54" width="1.27" layer="16"/>
-<wire x1="32.16659375" y1="26.63340625" x2="32.16659375" y2="18.06659375" width="1.27" layer="16"/>
+<wire x1="32.16659375" y1="26.23340625" x2="32.16659375" y2="18.06659375" width="1.27" layer="16"/>
 <wire x1="32.1" y1="18" x2="32.16659375" y2="18.06659375" width="1.27" layer="16"/>
 <wire x1="35.49" y1="12.48" x2="35.49" y2="14.61" width="1.27" layer="16"/>
@@
 <contactref element="JP7" pad="2"/>
 <contactref element="JP2" pad="5"/>
-<wire x1="11.285" y1="8.315" x2="11.285" y2="4.67" width="2" layer="16"/>
+<wire x1="11.285" y1="8.315" x2="11.185" y2="4.87" width="2" layer="16"/>
 <wire x1="6.84" y1="40.98" x2="6.84" y2="12.56" width="2" layer="16"/>
 <wire x1="6.84" y1="12.56" x2="7" y2="12.4" width="2" layer="16"/>
@@
 <contactref element="JP7" pad="3"/>
 <contactref element="JP2" pad="4"/>
-<wire x1="13.825" y1="4.67" x2="13.825" y2="9.975" width="2" layer="16"/>
+<wire x1="13.725" y1="4.87" x2="13.825" y2="9.975" width="2" layer="16"/>
 <wire x1="13.825" y1="9.975" x2="9.4" y2="14.4" width="2" layer="16"/>
 <wire x1="9.4" y1="14.4" x2="9.4" y2="41.06" width="2" layer="16"/>
@@
 <contactref element="JP10" pad="3"/>
 <wire x1="27.6" y1="12.3" x2="27.6" y2="12.929375" width="2" layer="16"/>
-<wire x1="23.17" y1="4.67" x2="21.445" y2="4.67" width="2" layer="16"/>
+<wire x1="23.17" y1="4.67" x2="21.345" y2="4.87" width="2" layer="16"/>
 <wire x1="25.95" y1="7.45" x2="23.17" y2="4.67" width="2" layer="16"/>
 <wire x1="25.95" y1="7.45" x2="27.6" y2="9.1" width="2" layer="16"/>
 <wire x1="27.6" y1="9.1" x2="27.6" y2="12.3" width="2" layer="16"/>
-<wire x1="18.905" y1="4.67" x2="21.445" y2="4.67" width="2" layer="16"/>
-<wire x1="21.83" y1="4.67" x2="21.445" y2="4.67" width="2" layer="16"/>
+<wire x1="18.805" y1="4.87" x2="21.345" y2="4.87" width="2" layer="16"/>
+<wire x1="21.83" y1="4.67" x2="21.345" y2="4.87" width="2" layer="16"/>
 <wire x1="22" y1="4.5" x2="21.83" y2="4.67" width="2" layer="16"/>
 <wire x1="22" y1="4.5" x2="21.615" y2="4.5" width="2" layer="16"/>
-<wire x1="21.615" y1="4.5" x2="21.445" y2="4.67" width="2" layer="16"/>
+<wire x1="21.615" y1="4.5" x2="21.345" y2="4.87" width="2" layer="16"/>
 <wire x1="11.92" y1="40.98" x2="11.92" y2="17.58" width="0.6096" layer="16"/>
 <wire x1="11.92" y1="17.58" x2="18.8" y2="10.7" width="0.6096" layer="16"/>
 <wire x1="18.8" y1="10.7" x2="18.8" y2="4.775" width="0.6096" layer="16"/>
-<wire x1="18.8" y1="4.775" x2="18.905" y2="4.67" width="0.6096" layer="16"/>
+<wire x1="18.8" y1="4.775" x2="18.805" y2="4.87" width="0.6096" layer="16"/>
 <contactref element="JP4" pad="2"/>
 <wire x1="28.73" y1="4.7" x2="28.7" y2="4.7" width="2" layer="16"/>
@@
 <contactref element="JP7" pad="5"/>
 <contactref element="JP2" pad="3"/>
-<wire x1="16.365" y1="4.67" x2="16.365" y2="9.565" width="1.27" layer="16"/>
+<wire x1="16.265" y1="4.87" x2="16.365" y2="9.565" width="1.27" layer="16"/>
 <wire x1="16.365" y1="9.565" x2="16.4" y2="9.6" width="1.27" layer="16"/>
 <via x="16.4" y="9.6" extent="1-16" drill="1"/>
@@
 <wire x1="27.6" y1="30.1" x2="27.6" y2="33.2" width="2" layer="16"/>
 <wire x1="27.6" y1="33.2" x2="29.2" y2="34.8" width="2" layer="16"/>
-<wire x1="29.2" y1="34.8" x2="29.2" y2="40.96" width="2" layer="16"/>
-<wire x1="29.2" y1="40.96" x2="29.14" y2="41.02" width="2" layer="16"/>
+<wire x1="29.2" y1="34.8" x2="28.9" y2="37.86" width="2" layer="16"/>
+<wire x1="28.9" y1="37.86" x2="28.94" y2="40.72" width="2" layer="16"/>
 <wire x1="25.06" y1="30.1" x2="27.6" y2="30.1" width="2" layer="16"/>
 </signal>
@@
 <contactref element="JP8" pad="3"/>
 <contactref element="JP11" pad="1"/>
-<wire x1="26.6" y1="39.34395625" x2="26.6" y2="41.02" width="2" layer="16"/>
+<wire x1="26.4" y1="39.24395625" x2="26.4" y2="40.72" width="2" layer="16"/>
 <wire x1="22.52" y1="30.1" x2="22.52" y2="32.56395625" width="2" layer="16"/>
-<wire x1="22.52" y1="32.56395625" x2="26.6" y2="39.34395625" width="2" layer="16"/>
+<wire x1="22.52" y1="32.56395625" x2="26.4" y2="39.24395625" width="2" layer="16"/>
 </signal>
 <signal name="+5V">
 <contactref element="JP8" pad="4"/>
 <contactref element="JP10" pad="1"/>
-<wire x1="24.06" y1="41.02" x2="19.7" y2="33.96" width="2" layer="16"/>
+<wire x1="23.86" y1="40.72" x2="19.7" y2="33.96" width="2" layer="16"/>
 <wire x1="19.7" y1="15.12" x2="22.52" y2="12.3" width="2" layer="16"/>
 <wire x1="19.7" y1="33.96" x2="19.7" y2="15.12" width="2" layer="16"/>
@@
 <contactref element="JP11" pad="5"/>
 <wire x1="32.68" y1="30.1" x2="32.68" y2="40.02" width="2" layer="16"/>
-<wire x1="32.68" y1="40.02" x2="31.68" y2="41.02" width="2" layer="16"/>
+<wire x1="32.68" y1="40.02" x2="31.48" y2="40.72" width="2" layer="16"/>
 </signal>
 <signal name="SW">
@@
 <wire x1="23.16" y1="8.46" x2="24.3" y2="9.6" width="1.016" layer="16"/>
 </signal>
+<signal name="N$6">
+<polygon width="0.1524" layer="16" isolate="1.6764">
+<vertex x="-0.5" y="44.2"/>
+<vertex x="52.4" y="44.2"/>
+<vertex x="51.8" y="-0.7"/>
+<vertex x="-0.7" y="-0.7"/>
+<vertex x="-0.7" y="-0.5"/>
+<vertex x="-1" y="-0.5"/>
+<vertex x="-1" y="42.3"/>
+</polygon>
+</signal>
 </signals>
