File: mukumiDevice/utility.sch (EAGLE design)
At the start: 11 parts

Commit message: 負電圧の信号を取るため、atmega328のPWM(analogWrite)とRCローパスを用いてVCC/2を生成し、それを抵抗(1.8kのやつ）で加算してからAD変換ポートにつなぐ
Parts:
- added JP3: (no value), pinhead:PINHD-1X8
- added JP4: (no value), pinhead:PINHD-1X2
Connections:
- net +5V: now also JP10.4, JP4.1
- net GND1: now also JP4.2
Changed lines of the file:
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@@
 <part name="JP10" library="pinhead" deviceset="PINHD-1X5" device=""/>
 <part name="JP11" library="pinhead" deviceset="PINHD-1X5" device=""/>
+<part name="JP3" library="pinhead" deviceset="PINHD-1X8" device=""/>
+<part name="JP4" library="pinhead" deviceset="PINHD-1X2" device=""/>
 </parts>
 <sheets>
@@
 <instance part="JP10" gate="A" x="154.94" y="96.52"/>
 <instance part="JP11" gate="A" x="134.62" y="96.52"/>
+<instance part="JP3" gate="A" x="152.4" y="73.66"/>
+<instance part="JP4" gate="G$1" x="147.32" y="-5.08"/>
 </instances>
 <busses>
@@
 <pinref part="JP10" gate="A" pin="3"/>
 </segment>
+<segment>
+<pinref part="JP4" gate="G$1" pin="2"/>
+<wire x1="144.78" y1="-5.08" x2="134.62" y2="-5.08" width="0.1524" layer="91"/>
+<label x="134.62" y="-5.08" size="1.778" layer="95"/>
+</segment>
 </net>
 <net name="VCC" class="0">
@@
 <pinref part="JP10" gate="A" pin="1"/>
 </segment>
-</net>
+<segment>
+<pinref part="JP4" gate="G$1" pin="1"/>
+<wire x1="144.78" y1="-2.54" x2="134.62" y2="-2.54" width="0.1524" layer="91"/>
+<label x="134.62" y="-2.54" size="1.778" layer="95"/>
+</segment>
+<segment>
+<wire x1="152.4" y1="93.98" x2="144.78" y2="93.98" width="0.1524" layer="91"/>
+<label x="144.78" y="93.98" size="1.778" layer="95"/>
+<pinref part="JP10" gate="A" pin="4"/>
+</segment>
+</net>
