File: mukumiDevice/utility_v2.brd (EAGLE design)
At the start: 51 x 43.6 mm, 13 parts

Commit message: 部品表に0ohm抵抗が抜けていたのを訂正、メイン基板のサイズに合わせてユーティリティ基板のピンの位置、サイズの変更
Parts:
- removed CURRENT_OUT, MESURE_VOL: STEREO3.5MM, audiojack:3.5MM
- removed JP1, JP10, JP11: (no value), pinhead:1X05
- removed JP4: (no value), pinhead:1X02
- removed JP7: (no value), pinhead:1X06
- removed JP8: (no value), pinhead:1X04
- removed JP9: (no value), pinhead:1X01
- removed R1: (no value), rcl:0204/5
- removed R2: (no value), rcl:0204/7
- added SV1: (no value), con-lstb:MA05-1
- added SV2: (no value), con-lstb:MA06-1
- JP2: device pinhead:1X06 -> pinhead:1X04
- JP3: device pinhead:1X08 -> pinhead:2X03
- moved JP3 57.7 mm to (4.14, 10.7)
- moved JP2 38.2 mm to (27.7, 40.7), turned to 0 degrees
Connections:
- removed net +12V: JP11.1, JP8.3
- removed net +5V: JP10.1, JP10.4, JP4.1, JP8.4
- removed net -12V: JP11.5, JP8.1
- removed net DTR: JP2.6
- removed net GND1: JP10.3, JP2.1, JP2.2, JP4.2, JP7.4
- removed net GND2: JP11.2, JP11.3, JP8.2
- removed net N$1: CURRENT_OUT.P$1, JP1.3, MESURE_VOL.P$1, R1.2, R2.1
- removed net N$2: CURRENT_OUT.P$4, JP1.1
- removed net N$3: CURRENT_OUT.P$3, JP1.5
- removed net N$4: JP1.2, MESURE_VOL.P$4
- removed net N$5: JP1.4, MESURE_VOL.P$3
- removed net N$7: CURRENT_OUT.P$2, MESURE_VOL.P$2, R1.1
- removed net N$8: CURRENT_OUT.P$5, MESURE_VOL.P$5, R2.2
- removed net RXD: JP2.5, JP7.2
- removed net SW: JP10.2, JP10.5, JP9.1
- removed net TXD: JP2.4, JP7.3
- removed net VCC: JP2.3, JP7.5
- new net AGND: SV1.3
- new net DENKYOKU1: SV1.4
- new net DENKYOKU2: SV1.2
- new net I1: SV1.5
- new net I2: SV1.1
Routing:
- net N$1: track 63.7 -> 0.00 mm
- net GND1: track 58.7 -> 0.00 mm
- net +5V: track 53.3 -> 0.00 mm
- net N$3: track 43.5 -> 0.00 mm
- net TXD: track 38.3 -> 0.00 mm
- net RXD: track 38.3 -> 0.00 mm
- net VCC: track 37.2 -> 0.00 mm, vias 2 -> 0
- net N$2: track 30.5 -> 0.00 mm
- net N$8: track 26.0 -> 0.00 mm
- net N$5: track 21.1 -> 0.00 mm
- net N$7: track 20.6 -> 0.00 mm
- net SW: track 17.9 -> 0.00 mm, vias 2 -> 0
- net GND2: track 14.1 -> 0.00 mm
- net +12V: track 12.1 -> 0.00 mm
- net -12V: track 11.3 -> 0.00 mm
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Other:
- board size 51 x 43.6 mm -> 49.2 x 43.9 mm
- board text added: "D1"
- board text added: "D2"
- board text added: "D3"
- board text added: "D4"
- board text added: "IC10"
- board text added: "IC14"
- board text added: "IC9"
- board text added: "SJ1"
- board text added: "SJ2"
- board text added: "SJ4"
- board text added: "SJ5"
- board text added: "VR1"
