File: mukumiDevice/utility_for_ad633.brd (EAGLE design)
At the start: 51 x 43.6 mm, 13 parts

Commit message: ユーティリティ基板の配線の調整とガーバーデータ出力
Parts:
- removed JP10, JP11: (no value), pinhead:1X05
- removed JP4: (no value), pinhead:1X02
- removed JP9: (no value), pinhead:1X01
- added C1, C2, C3, C4: (no value), rcl:E2-5
- added C5, C6, C7, C8: (no value), rcl:C2012
- added IC1: (no value), v-reg:78XXS
- added IC2: (no value), v-reg:79XXS
- JP3: device pinhead:1X08 -> pinhead:1X03
- moved JP3 37.2 mm to (27.7, 4.60), turned to 0 degrees
- moved JP8 0.36 mm to (27.7, 40.7)
- moved JP1 0.32 mm to (41.2, 40.7)
- moved JP2 0.22 mm to (15.0, 4.87)
Connections:
- removed net +12V: JP11.1, JP8.3
- removed net -12V: JP11.5, JP8.1
- removed net SW: JP10.2, JP10.5, JP9.1
- new net -5V: C3.-, C8.2, IC2.OUT, JP8.1
- new net VIN+: C1.+, C6.1, IC1.IN, JP3.1
- new net VIN-: C2.-, C5.2, IC2.IN, JP3.2
- net +5V: now also C4.+, C7.1, IC1.OUT, JP8.3; no longer JP10.1, JP10.4, JP4.1
- net GND1: no longer JP10.3, JP4.2
- net GND2: now also C1.-, C2.+, C3.+, C4.-, C5.1, C6.2, C7.2, C8.1, IC1.GND, IC2.GND, JP3.3; no longer JP11.2, JP11.3
Routing:
- net GND2: track 14.1 -> 70.4 mm
- net -5V: track 0.00 -> 38.8 mm, vias 0 -> 2
- net +5V: track 53.3 -> 14.8 mm
- net VIN+: track 0.00 -> 34.8 mm
- net VIN-: track 0.00 -> 20.0 mm
- net SW: track 17.9 -> 0.00 mm, vias 2 -> 0
- net GND1: track 58.7 -> 41.3 mm
- net +12V: track 12.1 -> 0.00 mm
- net -12V: track 11.3 -> 0.00 mm
- net N$8: track 26.0 -> 25.0 mm
- added copper zone on layer 16, net N$6
