File: mukumiDevice/mukumi_add_adc.brd (EAGLE design)
At the start: 49.2 x 49.6 mm, 151 parts, among them IC1 AD835, IC10 NJM2884, IC11 AD9834, IC12 AD9834, IC13 SIT8002B, IC14 NJM074V, IC2 AD835, IC5 NJM074V, IC6 NJM074V, IC7 NJM074V, IC8 NJM074V, IC9 NJM2884

Commit message: ACカップリングコンデンサをPMLCAPへ変更とadc通信用i2cパスにプルアップ抵抗の追加
Parts:
- added R52, R53: 10k, rcl:R0402
- C2: value 0.47u -> (none); device rcl:PANASONIC_B -> rcl:C1206
- C23, C40: device rcl:PANASONIC_B -> rcl:C1812K
- C3, C4, C56, C57, C58, C59: device rcl:PANASONIC_B -> rcl:C1206
- moved C50 4.67 mm to (25.4, 31.0), turned to 90 degrees
- moved D3 4.44 mm to (24.4, 19.1), turned to 90 degrees
- moved C23 4.30 mm to (35.0, 35.2), turned to 90 degrees
- moved C49 4.07 mm to (23.6, 34.8)
- moved R26 3.06 mm to (18.2, 33.6)
- moved C40 2.83 mm to (34.8, 25.6), turned to 180 degrees
- moved C4 2.80 mm to (17.5, 29.9), turned to 90 degrees
- moved C24 2.40 mm to (11.2, 40.4)
- moved C38 2.40 mm to (41.2, 37.6)
- moved JP2 2.40 mm to (27.7, 40.7)
- moved R35 2.40 mm to (36.5, 37.1)
- moved SV1 2.40 mm to (41.3, 40.7)
- moved C1 2.40 mm to (25.9, 31.3)
- moved C10 2.40 mm to (5.55, 34.4)
- moved C12 2.40 mm to (30.1, 33.5)
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Connections:
- net 3.3V_DDS: now also R52.2, R53.1
- net A1: now also C40.1; no longer C40.+
- net AGND: now also C56.2, C58.2; no longer C56.-, C58.-
- net DDS_OUT1: now also C3.1; no longer C3.+
- net DDS_OUT2: now also C4.1; no longer C4.+
- net N$2: now also C56.1; no longer C56.+
- net N$3: now also C58.1; no longer C58.+
- net N$4: now also C57.1; no longer C57.+
- net N$41: now also C23.2; no longer C23.-
- net N$45: now also C4.2; no longer C4.-
- net N$46: now also C40.2; no longer C40.-
- net N$54: now also C2.1; no longer C2.+
- net N$55: now also C2.2; no longer C2.-
- net N$56: now also C23.1; no longer C23.+
- net N$6: now also C59.1; no longer C59.+
- net N$64: now also C3.2; no longer C3.-
- net SCL_AD: now also R52.1
- net SDA_AD: now also R53.2
- net SIG*COS: now also C57.2; no longer C57.-
- net SIG*SIN: now also C59.2; no longer C59.-
Routing:
- net GND: track 206.5 -> 214.8 mm
- net AGND: track 392.9 -> 400.5 mm
- net 3.3V_DDS: track 133.6 -> 140.9 mm
- net AOUT2: track 40.8 -> 47.9 mm
- net AOUT1: track 45.0 -> 50.9 mm
- net +5V: track 128.0 -> 133.7 mm
- net N$48: track 14.5 -> 19.8 mm
- net SIG*SIN: track 43.7 -> 48.7 mm, vias 3 -> 4
- net N$44: track 20.4 -> 25.4 mm
- net -5V: track 111.8 -> 116.3 mm
- net DDS_OUT2: track 5.51 -> 9.89 mm
- net SIN: track 32.8 -> 37.1 mm
- net N$78: track 10.7 -> 14.2 mm
- net N$6: track 19.2 -> 16.1 mm, vias 1 -> 0
- net SIG: track 11.9 -> 14.9 mm
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
Commit message: 乗算器をAD865またはAD633に選択可能に
Parts:
- added R54, R55, R58, R73: 0, rcl:R0402
- C2: value (none) -> 0.47u; device rcl:C1206 -> rcl:C1812K
- C3, C4, C56, C57, C58, C59: device rcl:C1206 -> rcl:C1812K
- R13: value 560 -> 5.6k
- R20: value 680 -> 6.8k
- R23: value 360 -> 3.6k
- R27: value 1k -> 7.5k
- R28: value 1k -> 11k
- R59, R60, R61, R62, R63, R64, R65, R66, R67, R68, R69, R70, R71, R72: value 560a -> 4.7k
- moved R53 8.69 mm to (11.0, 7.60)
- moved C45 2.25 mm to (35.1, 5.36), turned to 270 degrees
- moved C59 2.24 mm to (46.8, 3.50), flipped to the bottom, turned to 90 degrees
- moved R52 2.13 mm to (19.3, 10.7)
- moved C56 2.12 mm to (26.9, 15.4), turned to 0 degrees
- moved C2 1.43 mm to (46.5, 27.1)
- moved C43 1.36 mm to (41.0, 4.84)
- moved C7 1.35 mm to (21.2, 9.60)
Connections:
- new net N$12: R54.1, R55.1, SJ3.2
- new net N$5: IC1.8, IC2.8, R54.2, R73.2
- net 3.3V_DDS: no longer R52.2, R53.1
- net 3.3V_MC: now also R52.2, R53.2
- net AGND: now also R58.1, R73.1; no longer IC1.8, IC2.8
- net SCL_AD: now also R53.1; no longer R52.1
- net SDA_AD: now also R52.1; no longer R53.2
- net SIG_: now also R55.2, R58.2; no longer SJ3.2
Routing:
- net N$5: track 0.00 -> 33.1 mm
- net 3.3V_MC: track 110.0 -> 120.3 mm
- net AGND: track 400.5 -> 404.8 mm, vias 26 -> 27
- net 3.3V_DDS: track 140.9 -> 136.7 mm
- net N$12: track 0.00 -> 4.04 mm
- net SIG*SIN: track 48.7 -> 45.0 mm, vias 4 -> 3
- net N$6: track 16.1 -> 19.7 mm, vias 0 -> 1
- net SIG_: track 28.4 -> 25.3 mm, vias 1 -> 0
- net GND: track 214.8 -> 212.3 mm
- net SIG*COS: track 20.4 -> 19.2 mm
- net N$55: track 9.88 -> 11.0 mm
- net DDS_OUT1: track 16.0 -> 15.0 mm
- net N$24: track 9.89 -> 10.6 mm
- net +5V: track 133.7 -> 134.3 mm
- net N$45: track 2.38 -> 1.73 mm
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
Commit message: 抵抗の値調整 部品表の出力、P板用部品表の追加
Parts:
- removed C1: 0.1u, rcl:C0402
- added C8: 0.1u, rcl:C0402
- C2, C3, C4: device rcl:C1812K -> rcl:C1206
- C56, C57, C58, C59: value (none) -> 0.47u; device rcl:C1812K -> rcl:C1206
- R37, R38: value 56 -> 5.6k
- R39, R40: value 560 -> 56k
- R42: value 62a -> 6.2k
- R43: value 560a -> 56k
- R44, R46, R47, R48, R50, R51, R56, R57: value 560a -> 560
- moved C11 5.34 mm to (25.7, 31.3), flipped to the top, turned to 90 degrees
- moved C56 0.30 mm to (27.2, 15.4)
- moved R31 0.20 mm to (33.5, 28.2)
- moved C57 0.20 mm to (34.1, 17.7)
- renumbered U$1 to IC3
Connections:
- net +5V: now also C8.1; no longer C11.1
- net AGND: now also C11.1, C8.2; no longer C1.1, C11.2
- net N$61: now also C11.2; no longer C1.2
Routing:
- net AGND: track 404.8 -> 406.1 mm
- net DDS_OUT1: track 15.0 -> 16.0 mm
- net SIG*COS: track 19.2 -> 20.0 mm
- net N$45: track 1.73 -> 2.38 mm
- net N$55: track 11.0 -> 11.6 mm

Commit message: 実装図（シルク面）の調整
Parts:
- IC3: value AD3422 -> MCP3422
- moved R33 0.10 mm to (31.1, 35.9)
Routing:
- net SIG*SIN: track 44.9 -> 43.1 mm
- net N$47: track 7.29 -> 6.07 mm
- net N$55: track 11.6 -> 10.8 mm
Other:
- board size 49.2 x 49.6 mm -> 49.2 x 43.9 mm
- board text added: "IC10"
- board text added: "IC9"
- board text added: "SJ1"
- board text added: "SJ2"
- board text added: "SJ4"
- board text added: "SJ5"

Commit message: 配線の調整
Parts:
- moved C7 1.33 mm to (20.9, 8.30), turned to 270 degrees
- moved D4 0.60 mm to (22.0, 15.2)
- moved R57 0.32 mm to (34.1, 8.70)
Routing:
- net 3.3V_DDS: track 136.8 -> 163.4 mm
- net N$44: track 25.1 -> 17.0 mm
- net AGND: track 406.3 -> 412.4 mm
- net +5V: track 134.6 -> 130.6 mm
- net AOUT1: track 50.4 -> 48.1 mm
- net GND: track 212.3 -> 210.2 mm
- net N$64: track 8.97 -> 6.86 mm
- net 3.3V_MC: track 120.3 -> 118.8 mm
- net N$91: track 12.8 -> 11.3 mm
- net N$4: track 12.2 -> 10.9 mm
- net +BATTERY: track 61.4 -> 60.3 mm
- net SIG*SIN: track 43.1 -> 42.3 mm
- net SIN: track 37.2 -> 36.4 mm
- net N$3: track 13.2 -> 12.5 mm
- net -5V: track 116.2 -> 116.8 mm
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
Commit message: 加算回路で使用するオペアンプの電源の±が逆につながっていたのを修正
Connections:
- net +5V: now also IC14.4; no longer IC14.11
- net -5V: now also IC14.11; no longer IC14.4
Routing:
- net +5V: track 130.6 -> 128.3 mm
- net AGND: track 412.4 -> 411.0 mm
- net -5V: track 116.8 -> 116.0 mm, vias 6 -> 7

Commit message: 部品表に0ohm抵抗が抜けていたのを訂正、メイン基板のサイズに合わせてユーティリティ基板のピンの位置、サイズの変更
Parts:
- C2, C3, C4, C56, C57, C58, C59: value 0.47u -> 1u
Changed lines of the file:
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@@
 <attribute name="VALUE" x="47.135" y="8.995" size="1.27" layer="28" rot="MR0"/>
 </element>
-<element name="C2" library="rcl" library_urn="urn:adsk.eagle:library:334" package="C1206" package3d_urn="urn:adsk.eagle:package:23618/2" value="0.47u" x="46.5" y="27.1" rot="MR90">
+<element name="C2" library="rcl" library_urn="urn:adsk.eagle:library:334" package="C1206" package3d_urn="urn:adsk.eagle:package:23618/2" value="1u" x="46.5" y="27.1" rot="MR90">
 <attribute name="SPICEPREFIX" value="C" x="46.5" y="27.1" size="1.778" layer="28" rot="MR90" display="off"/>
 </element>
-<element name="C3" library="rcl" library_urn="urn:adsk.eagle:library:334" package="C1206" package3d_urn="urn:adsk.eagle:package:23618/2" value="0.47u" x="20.7" y="19.4" rot="MR270">
+<element name="C3" library="rcl" library_urn="urn:adsk.eagle:library:334" package="C1206" package3d_urn="urn:adsk.eagle:package:23618/2" value="1u" x="20.7" y="19.4" rot="MR270">
 <attribute name="SPICEPREFIX" value="C" x="20.7" y="19.4" size="1.778" layer="28" rot="MR270" display="off"/>
 </element>
-<element name="C4" library="rcl" library_urn="urn:adsk.eagle:library:334" package="C1206" package3d_urn="urn:adsk.eagle:package:23618/2" value="0.47u" x="17.5" y="29.9" rot="MR90">
+<element name="C4" library="rcl" library_urn="urn:adsk.eagle:library:334" package="C1206" package3d_urn="urn:adsk.eagle:package:23618/2" value="1u" x="17.5" y="29.9" rot="MR90">
 <attribute name="SPICEPREFIX" value="C" x="17.5" y="29.9" size="1.778" layer="28" rot="MR90" display="off"/>
 </element>
@@
 <attribute name="SPICEPREFIX" value="C" x="34.8" y="25.6" size="1.778" layer="28" rot="MR180" display="off"/>
 </element>
-<element name="C56" library="rcl" library_urn="urn:adsk.eagle:library:334" package="C1206" package3d_urn="urn:adsk.eagle:package:23618/2" value="0.47u" x="27.2" y="15.4" rot="MR0">
+<element name="C56" library="rcl" library_urn="urn:adsk.eagle:library:334" package="C1206" package3d_urn="urn:adsk.eagle:package:23618/2" value="1u" x="27.2" y="15.4" rot="MR0">
 <attribute name="SPICEPREFIX" value="C" x="27.2" y="15.4" size="1.778" layer="28" rot="MR0" display="off"/>
 </element>
-<element name="C57" library="rcl" library_urn="urn:adsk.eagle:library:334" package="C1206" package3d_urn="urn:adsk.eagle:package:23618/2" value="0.47u" x="34.1" y="17.7" smashed="yes" rot="MR270">
+<element name="C57" library="rcl" library_urn="urn:adsk.eagle:library:334" package="C1206" package3d_urn="urn:adsk.eagle:package:23618/2" value="1u" x="34.1" y="17.7" smashed="yes" rot="MR270">
 <attribute name="NAME" x="32.83" y="18.97" size="1.27" layer="26" rot="MR270"/>
 <attribute name="SPICEPREFIX" value="C" x="34.1" y="17.7" size="1.778" layer="28" rot="MR270" display="off"/>
 <attribute name="VALUE" x="36.64" y="18.97" size="1.27" layer="28" rot="MR270"/>
 </element>
-<element name="C58" library="rcl" library_urn="urn:adsk.eagle:library:334" package="C1206" package3d_urn="urn:adsk.eagle:package:23618/2" value="0.47u" x="26.8" y="4.5" smashed="yes" rot="MR90">
+<element name="C58" library="rcl" library_urn="urn:adsk.eagle:library:334" package="C1206" package3d_urn="urn:adsk.eagle:package:23618/2" value="1u" x="26.8" y="4.5" smashed="yes" rot="MR90">
 <attribute name="NAME" x="27.97" y="2.53" size="1.27" layer="26" rot="MR90"/>
 <attribute name="SPICEPREFIX" value="C" x="26.8" y="4.5" size="1.778" layer="28" rot="MR90" display="off"/>
 <attribute name="VALUE" x="24.26" y="3.23" size="1.27" layer="28" rot="MR90"/>
 </element>
-<element name="C59" library="rcl" library_urn="urn:adsk.eagle:library:334" package="C1206" package3d_urn="urn:adsk.eagle:package:23618/2" value="0.47u" x="46.8" y="3.5" rot="MR90">
+<element name="C59" library="rcl" library_urn="urn:adsk.eagle:library:334" package="C1206" package3d_urn="urn:adsk.eagle:package:23618/2" value="1u" x="46.8" y="3.5" rot="MR90">
 <attribute name="SPICEPREFIX" value="C" x="46.8" y="3.5" size="1.778" layer="28" rot="MR90" display="off"/>
 </element>

Commit message: P板からの指摘点を修正、ad633用ユーティリティ基板の作成
Parts:
- R44, R48: value 560 -> 4.7k
- moved C7 0.30 mm to (20.6, 8.30)
- moved C13 0.10 mm to (3.68, 31.7)
Routing:
- net AGND: track 411.0 -> 413.4 mm
