File: mukumiDevice/mukumi_add_adc.sch (EAGLE design)
At the start: 157 parts, among them IC1 AD835, IC10 NJM2884, IC11 AD9834, IC12 AD9834, IC13 SIT8002B, IC14 NJM074V, IC2 AD835, IC5 NJM074V, IC6 NJM074V, IC7 NJM074V, IC8 NJM074V, IC9 NJM2884

Commit message: 抵抗の値調整 部品表の出力、P板用部品表の追加
Parts:
- removed C1: 0.1u, rcl:C-EUC0402
- added C8: 0.1u, rcl:C-EUC0402
- C2, C3, C4: device rcl:C-EUC1812K -> rcl:C-EUC1206
- C56, C57, C58, C59: value (none) -> 0.47u; device rcl:C-EUC1812K -> rcl:C-EUC1206
- R37, R38: value 56 -> 5.6k
- R39, R40: value 560 -> 56k
- R42: value 62a -> 6.2k
- R43: value 560a -> 56k
- R44, R46, R47, R48, R50, R51, R56, R57: value 560a -> 560
- renumbered U$1 to IC3
Connections:
- net +5V: now also C8.1; no longer C11.1
- net AGND: now also C11.1, C8.2; no longer C1.1, C11.2
- net N$61: now also C11.2; no longer C1.2
Other:
- moved on the sheet: C11

Commit message: 実装図（シルク面）の調整
Parts:
- IC3: value AD3422 -> MCP3422; device ad849x:AD3422 -> ad849x:MCP3422
Changed lines of the file:
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@@
 <part name="C5" library="rcl" deviceset="C-EU" device="C0402" value="0.1u"/>
 <part name="C6" library="rcl" deviceset="C-EU" device="C0402" value="0.1u"/>
-<part name="IC3" library="ad849x" deviceset="AD3422" device=""/>
+<part name="IC3" library="ad849x" deviceset="MCP3422" device=""/>
 <part name="GND29" library="supply1" deviceset="AGND" device=""/>
 <part name="GND30" library="supply1" deviceset="AGND" device=""/>

Commit message: 配線の調整
Changed lines of the file:
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@@
 <pinref part="R54" gate="G$1" pin="1"/>
 <pinref part="R55" gate="G$1" pin="1"/>
+<junction x="12.7" y="134.62"/>
 </segment>
 </net>

Commit message: 加算回路で使用するオペアンプの電源の±が逆につながっていたのを修正
Connections:
- net +5V: now also IC14G$1.V+; no longer IC14G$1.V-
- net -5V: now also IC14G$1.V-; no longer IC14G$1.V+
Changed lines of the file:
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@@
 <part name="R62" library="rcl" deviceset="R-EU_" device="R0402" value="4.7k"/>
 <part name="R63" library="rcl" deviceset="R-EU_" device="R0402" value="4.7k"/>
-<part name="P+1" library="supply1" deviceset="+5V" device=""/>
-<part name="P-1" library="supply1" deviceset="-5V" device=""/>
 <part name="GND41" library="supply1" deviceset="AGND" device=""/>
 <part name="GND42" library="supply1" deviceset="AGND" device=""/>
@@
 <part name="C8" library="rcl" deviceset="C-EU" device="C0402" value="0.1u"/>
 <part name="C11" library="rcl" deviceset="C-EU" device="C0402" value="0.1u"/>
+<part name="P+1" library="supply1" deviceset="+5V" device=""/>
+<part name="P-1" library="supply1" deviceset="-5V" device=""/>
 </parts>
 <sheets>
@@
 <instance part="R62" gate="G$1" x="269.24" y="88.9"/>
 <instance part="R63" gate="G$1" x="284.48" y="99.06"/>
-<instance part="P+1" gate="1" x="238.76" y="99.06"/>
-<instance part="P-1" gate="1" x="238.76" y="78.74"/>
 <instance part="GND41" gate="VR1" x="215.9" y="83.82"/>
 <instance part="GND42" gate="VR1" x="271.78" y="81.28"/>
@@
 <instance part="R58" gate="G$1" x="20.32" y="129.54"/>
 <instance part="R73" gate="G$1" x="20.32" y="124.46"/>
+<instance part="P+1" gate="1" x="246.38" y="76.2" rot="R270"/>
+<instance part="P-1" gate="1" x="246.38" y="101.6" rot="R90"/>
 </instances>
 <busses>
@@
 </segment>
 <segment>
-<pinref part="IC14" gate="G$1" pin="V-"/>
+<pinref part="IC14" gate="G$1" pin="V+"/>
 <pinref part="P+1" gate="1" pin="+5V"/>
+<wire x1="243.84" y1="76.2" x2="238.76" y2="81.28" width="0.1524" layer="91"/>
 </segment>
 </net>
@@
 </segment>
 <segment>
-<pinref part="IC14" gate="G$1" pin="V+"/>
+<pinref part="IC14" gate="G$1" pin="V-"/>
 <pinref part="P-1" gate="1" pin="-5V"/>
-</segment>
-</net>
+<wire x1="243.84" y1="101.6" x2="238.76" y2="96.52" width="0.1524" layer="91"/>
+</segment>
+</net>

Commit message: 部品表に0ohm抵抗が抜けていたのを訂正、メイン基板のサイズに合わせてユーティリティ基板のピンの位置、サイズの変更
Parts:
- C2, C3, C4, C56, C57, C58, C59: value 0.47u -> 1u
Changed lines of the file:
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@@
 <part name="R72" library="rcl" deviceset="R-EU_" device="R0402" value="4.7k"/>
 <part name="GND44" library="supply1" deviceset="AGND" device=""/>
-<part name="C2" library="rcl" library_urn="urn:adsk.eagle:library:334" deviceset="C-EU" device="C1206" package3d_urn="urn:adsk.eagle:package:23618/2" value="0.47u"/>
-<part name="C3" library="rcl" library_urn="urn:adsk.eagle:library:334" deviceset="C-EU" device="C1206" package3d_urn="urn:adsk.eagle:package:23618/2" value="0.47u"/>
-<part name="C4" library="rcl" library_urn="urn:adsk.eagle:library:334" deviceset="C-EU" device="C1206" package3d_urn="urn:adsk.eagle:package:23618/2" value="0.47u"/>
+<part name="C2" library="rcl" library_urn="urn:adsk.eagle:library:334" deviceset="C-EU" device="C1206" package3d_urn="urn:adsk.eagle:package:23618/2" value="1u"/>
+<part name="C3" library="rcl" library_urn="urn:adsk.eagle:library:334" deviceset="C-EU" device="C1206" package3d_urn="urn:adsk.eagle:package:23618/2" value="1u"/>
+<part name="C4" library="rcl" library_urn="urn:adsk.eagle:library:334" deviceset="C-EU" device="C1206" package3d_urn="urn:adsk.eagle:package:23618/2" value="1u"/>
 <part name="C23" library="rcl" library_urn="urn:adsk.eagle:library:334" deviceset="C-EU" device="C1812K" package3d_urn="urn:adsk.eagle:package:23686/2" value="4.7u"/>
 <part name="C40" library="rcl" library_urn="urn:adsk.eagle:library:334" deviceset="C-EU" device="C1812K" package3d_urn="urn:adsk.eagle:package:23686/2" value="4.7u"/>
-<part name="C56" library="rcl" library_urn="urn:adsk.eagle:library:334" deviceset="C-EU" device="C1206" package3d_urn="urn:adsk.eagle:package:23618/2" value="0.47u"/>
-<part name="C57" library="rcl" library_urn="urn:adsk.eagle:library:334" deviceset="C-EU" device="C1206" package3d_urn="urn:adsk.eagle:package:23618/2" value="0.47u"/>
-<part name="C58" library="rcl" library_urn="urn:adsk.eagle:library:334" deviceset="C-EU" device="C1206" package3d_urn="urn:adsk.eagle:package:23618/2" value="0.47u"/>
-<part name="C59" library="rcl" library_urn="urn:adsk.eagle:library:334" deviceset="C-EU" device="C1206" package3d_urn="urn:adsk.eagle:package:23618/2" value="0.47u"/>
+<part name="C56" library="rcl" library_urn="urn:adsk.eagle:library:334" deviceset="C-EU" device="C1206" package3d_urn="urn:adsk.eagle:package:23618/2" value="1u"/>
+<part name="C57" library="rcl" library_urn="urn:adsk.eagle:library:334" deviceset="C-EU" device="C1206" package3d_urn="urn:adsk.eagle:package:23618/2" value="1u"/>
+<part name="C58" library="rcl" library_urn="urn:adsk.eagle:library:334" deviceset="C-EU" device="C1206" package3d_urn="urn:adsk.eagle:package:23618/2" value="1u"/>
+<part name="C59" library="rcl" library_urn="urn:adsk.eagle:library:334" deviceset="C-EU" device="C1206" package3d_urn="urn:adsk.eagle:package:23618/2" value="1u"/>
 <part name="C5" library="rcl" deviceset="C-EU" device="C0402" value="0.1u"/>
 <part name="C6" library="rcl" deviceset="C-EU" device="C0402" value="0.1u"/>

Commit message: P板からの指摘点を修正、ad633用ユーティリティ基板の作成
Parts:
- R44, R48: value 560 -> 4.7k
Changed lines of the file:
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@@
 <part name="GND27" library="supply1" deviceset="AGND" device=""/>
 <part name="GND28" library="supply1" deviceset="AGND" device=""/>
-<part name="R44" library="rcl" deviceset="R-EU_" device="R0402" value="560"/>
-<part name="R48" library="rcl" deviceset="R-EU_" device="R0402" value="560"/>
+<part name="R44" library="rcl" deviceset="R-EU_" device="R0402" value="4.7k"/>
+<part name="R48" library="rcl" deviceset="R-EU_" device="R0402" value="4.7k"/>
 <part name="R45" library="rcl" deviceset="R-EU_" device="R0402" value="11k"/>
 <part name="R49" library="rcl" deviceset="R-EU_" device="R0402" value="11k"/>
@@
 <instance part="GND68" gate="VR1" x="7.62" y="63.5"/>
 <instance part="P+31" gate="1" x="-243.84" y="81.28" rot="R90"/>
-<instance part="P-14" gate="1" x="-243.84" y="66.04" rot="R270"/>
+<instance part="P-14" gate="1" x="-246.38" y="66.04" rot="R270"/>
 <instance part="SV1" gate="G$1" x="-119.38" y="38.1"/>
 <instance part="P+3" gate="1" x="-274.32" y="25.4"/>
@@
 <pinref part="P-14" gate="1" pin="-5V"/>
 <pinref part="IC7" gate="G$1" pin="V-"/>
-<junction x="-241.3" y="66.04"/>
-</segment>
-<segment>
+<wire x1="-243.84" y1="66.04" x2="-241.3" y2="66.04" width="0.1524" layer="91"/>
+</segment>
+<segment>
